Commit message: param command doesn't seem to be an option in ros2, so python use is mandated now

File: src/drqp_description/urdf/dr_qp.urdf.xacro (robot description, xacro)
@@ -9,5 +9,5 @@
   </xacro:if>
   <material name="drqp_black">
-    <texture filename="package://drqp_descriptions/meshes/drqp_black.png"/>
+    <texture filename="package://drqp_description/meshes/drqp_black.png"/>
   </material>
   <xacro:macro name="leg" params="robot_name prefix x y yaw">
@@ -33,5 +33,5 @@
         <origin rpy="0 0 0" xyz="0 0 0"/>
         <geometry>
-          <mesh filename="package://drqp_descriptions/meshes/dr_qp_meshes/dr_qp_coxa_link.stl" scale="0.001 0.001 0.001"/>
+          <mesh filename="package://drqp_description/meshes/dr_qp_meshes/dr_qp_coxa_link.stl" scale="0.001 0.001 0.001"/>
         </geometry>
         <material name="drqp_black"/>
@@ -40,5 +40,5 @@
         <origin rpy="0 0 0" xyz="0 0 0"/>
         <geometry>
-          <mesh filename="package://drqp_descriptions/meshes/dr_qp_meshes/dr_qp_coxa_link.stl" scale="0.001 0.001 0.001"/>
+          <mesh filename="package://drqp_description/meshes/dr_qp_meshes/dr_qp_coxa_link.stl" scale="0.001 0.001 0.001"/>
         </geometry>
       </collision>
@@ -70,5 +70,5 @@
         <origin rpy="0 0 0" xyz="0 0 0"/>
         <geometry>
-          <mesh filename="package://drqp_descriptions/meshes/dr_qp_meshes/dr_qp_femur_link.stl" scale="0.001 0.001 0.001"/>
+          <mesh filename="package://drqp_description/meshes/dr_qp_meshes/dr_qp_femur_link.stl" scale="0.001 0.001 0.001"/>
         </geometry>
         <material name="drqp_black"/>
@@ -77,5 +77,5 @@
         <origin rpy="0 0 0" xyz="0 0 0"/>
         <geometry>
-          <mesh filename="package://drqp_descriptions/meshes/dr_qp_meshes/dr_qp_femur_link.stl" scale="0.001 0.001 0.001"/>
+          <mesh filename="package://drqp_description/meshes/dr_qp_meshes/dr_qp_femur_link.stl" scale="0.001 0.001 0.001"/>
         </geometry>
       </collision>
@@ -107,5 +107,5 @@
         <origin rpy="0 0 0" xyz="0 0 0"/>
         <geometry>
-          <mesh filename="package://drqp_descriptions/meshes/dr_qp_meshes/dr_qp_tibia_link.stl" scale="0.001 0.001 0.001"/>
+          <mesh filename="package://drqp_description/meshes/dr_qp_meshes/dr_qp_tibia_link.stl" scale="0.001 0.001 0.001"/>
         </geometry>
         <material name="drqp_black"/>
@@ -114,5 +114,5 @@
         <origin rpy="0 0 0" xyz="0 0 0"/>
         <geometry>
-          <mesh filename="package://drqp_descriptions/meshes/dr_qp_meshes/dr_qp_tibia_link.stl" scale="0.001 0.001 0.001"/>
+          <mesh filename="package://drqp_description/meshes/dr_qp_meshes/dr_qp_tibia_link.stl" scale="0.001 0.001 0.001"/>
         </geometry>
       </collision>
@@ -134,5 +134,5 @@
       <origin rpy="0 0 0" xyz="0 0 0"/>
       <geometry>
-        <mesh filename="package://drqp_descriptions/meshes/dr_qp_meshes/dr_qp_base_link.stl" scale="0.001 0.001 0.001"/>
+        <mesh filename="package://drqp_description/meshes/dr_qp_meshes/dr_qp_base_link.stl" scale="0.001 0.001 0.001"/>
       </geometry>
       <material name="drqp_black"/>
@@ -141,5 +141,5 @@
       <origin rpy="0 0 0" xyz="0 0 0"/>
       <geometry>
-        <mesh filename="package://drqp_descriptions/meshes/dr_qp_meshes/dr_qp_base_link.stl" scale="0.001 0.001 0.001"/>
+        <mesh filename="package://drqp_description/meshes/dr_qp_meshes/dr_qp_base_link.stl" scale="0.001 0.001 0.001"/>
       </geometry>
     </collision>

Commit message: address the base link conflict with KDL make py launch work with new urdf

File: src/drqp_description/urdf/dr_qp.urdf.xacro (robot description, xacro)
@@ -11,4 +11,7 @@
     <texture filename="package://drqp_description/meshes/drqp_black.png"/>
   </material>
+  <material name="drqp_black_tmp">
+    <color rgba="0.5 0.5 0.5 0.2" />
+  </material>
   <xacro:macro name="leg" params="robot_name prefix x y yaw">
     <joint name="${prefix}_coxa" type="revolute">
@@ -16,5 +19,5 @@
       <limit effort="3" lower="${radians(-55)}" upper="${radians(55)}" velocity="${pi}"/>
       <origin rpy="0 0 ${yaw}" xyz="${x} ${y} 0"/>
-      <parent link="${robot_name}/base_link"/>
+      <parent link="${robot_name}/base_center_link"/>
       <child link="${robot_name}/${prefix}_coxa_link"/>
       <dynamics friction="0.5"/>
@@ -33,5 +36,5 @@
         <origin rpy="0 0 0" xyz="0 0 0"/>
         <geometry>
-          <mesh filename="package://drqp_description/meshes/dr_qp_meshes/dr_qp_coxa_link.stl" scale="0.001 0.001 0.001"/>
+          <mesh filename="package://drqp_description/meshes/coxa_link.stl" />
         </geometry>
         <material name="drqp_black"/>
@@ -40,5 +43,5 @@
         <origin rpy="0 0 0" xyz="0 0 0"/>
         <geometry>
-          <mesh filename="package://drqp_description/meshes/dr_qp_meshes/dr_qp_coxa_link.stl" scale="0.001 0.001 0.001"/>
+          <mesh filename="package://drqp_description/meshes/coxa_link.stl" />
         </geometry>
       </collision>
@@ -49,4 +52,5 @@
       </inertial>
     </link>
+<!--
     <joint name="${prefix}_femur" type="revolute">
       <axis xyz="0 1 0"/>
@@ -70,5 +74,5 @@
         <origin rpy="0 0 0" xyz="0 0 0"/>
         <geometry>
-          <mesh filename="package://drqp_description/meshes/dr_qp_meshes/dr_qp_femur_link.stl" scale="0.001 0.001 0.001"/>
+          <mesh filename="package://drqp_description/meshes/femur_link.stl" />
         </geometry>
         <material name="drqp_black"/>
@@ -77,5 +81,5 @@
         <origin rpy="0 0 0" xyz="0 0 0"/>
         <geometry>
-          <mesh filename="package://drqp_description/meshes/dr_qp_meshes/dr_qp_femur_link.stl" scale="0.001 0.001 0.001"/>
+          <mesh filename="package://drqp_description/meshes/femur_link.stl" />
         </geometry>
       </collision>
@@ -107,5 +111,5 @@
         <origin rpy="0 0 0" xyz="0 0 0"/>
         <geometry>
-          <mesh filename="package://drqp_description/meshes/dr_qp_meshes/dr_qp_tibia_link.stl" scale="0.001 0.001 0.001"/>
+          <mesh filename="package://drqp_description/meshes/tibia_link.stl" />
         </geometry>
         <material name="drqp_black"/>
@@ -114,5 +118,5 @@
         <origin rpy="0 0 0" xyz="0 0 0"/>
         <geometry>
-          <mesh filename="package://drqp_description/meshes/dr_qp_meshes/dr_qp_tibia_link.stl" scale="0.001 0.001 0.001"/>
+          <mesh filename="package://drqp_description/meshes/tibia_link.stl" />
         </geometry>
       </collision>
@@ -128,18 +132,18 @@
       <child link="${robot_name}/${prefix}_foot_link"/>
     </joint>
-    <link name="${robot_name}/${prefix}_foot_link"/>
+    <link name="${robot_name}/${prefix}_foot_link"/> -->
   </xacro:macro>
-  <link name="$(arg robot_name)/base_link">
+  <link name="$(arg robot_name)/base_center_link">
     <visual>
-      <origin rpy="0 0 0" xyz="0 0 0"/>
+      <origin xyz="0 0 0" rpy="${pi/2} 0 ${pi}" />
       <geometry>
-        <mesh filename="package://drqp_description/meshes/dr_qp_meshes/dr_qp_base_link.stl" scale="0.001 0.001 0.001"/>
+        <mesh filename="package://drqp_description/meshes/body-simple.stl" />
       </geometry>
       <material name="drqp_black"/>
     </visual>
     <collision>
-      <origin rpy="0 0 0" xyz="0 0 0"/>
+      <origin xyz="0 0 0" rpy="${pi/2} 0 ${pi}" />
       <geometry>
-        <mesh filename="package://drqp_description/meshes/dr_qp_meshes/dr_qp_base_link.stl" scale="0.001 0.001 0.001"/>
+        <mesh filename="package://drqp_description/meshes/body-simple.stl" />
       </geometry>
     </collision>
@@ -150,17 +154,17 @@
     </inertial>
   </link>
-  <joint name="base_bottom" type="fixed">
-    <origin rpy="0 0 0" xyz="0 0 -0.033"/>
-    <parent link="$(arg robot_name)/base_link"/>
-    <child link="$(arg robot_name)/base_bottom_link"/>
-  </joint>
   <link name="$(arg robot_name)/base_bottom_link">
   </link>
-  <xacro:leg robot_name="$(arg robot_name)" prefix="right_front" x="0.125" y="-0.065" yaw="${-pi/4}"/>
-  <xacro:leg robot_name="$(arg robot_name)" prefix="right_middle" x="0" y="-0.1" yaw="${-pi/2}"/>
-  <xacro:leg robot_name="$(arg robot_name)" prefix="right_back" x="-0.125" y="-0.065" yaw="${-3*pi/4}"/>
-  <xacro:leg robot_name="$(arg robot_name)" prefix="left_front" x="0.125" y="0.065" yaw="${pi/4}"/>
-  <xacro:leg robot_name="$(arg robot_name)" prefix="left_middle" x="0" y="0.1" yaw="${pi/2}"/>
-  <xacro:leg robot_name="$(arg robot_name)" prefix="left_back" x="-0.125" y="0.065" yaw="${3*pi/4}"/>
+  <joint name="base_bottom" type="fixed">
+    <origin rpy="0 0 0" xyz="0 0 0.033"/>
+    <child link="$(arg robot_name)/base_center_link"/>
+    <parent link="$(arg robot_name)/base_bottom_link"/>
+  </joint>
+  <xacro:leg robot_name="$(arg robot_name)" prefix="right_front" x="0.11692" y="-0.06387" yaw="${-pi/4}"/>
+  <xacro:leg robot_name="$(arg robot_name)" prefix="right_middle" x="0" y="-0.103" yaw="${-pi/2}"/>
+  <xacro:leg robot_name="$(arg robot_name)" prefix="right_back" x="-0.11692" y="-0.06387" yaw="${-3*pi/4}"/>
+  <xacro:leg robot_name="$(arg robot_name)" prefix="left_front" x="0.11692" y="0.06387" yaw="${pi/4}"/>
+  <xacro:leg robot_name="$(arg robot_name)" prefix="left_middle" x="0" y="0.103" yaw="${pi/2}"/>
+  <xacro:leg robot_name="$(arg robot_name)" prefix="left_back" x="-0.11692" y="0.06387" yaw="${3*pi/4}"/>
   <xacro:if value="${urdf_loc != ''}">
     <xacro:include filename="${urdf_loc}"/>

Commit message: add servos

File: src/drqp_description/urdf/dr_qp.urdf.xacro (robot description, xacro)
@@ -15,9 +15,34 @@
   </material>
   <xacro:macro name="leg" params="robot_name prefix x y yaw">
+    <joint name="${prefix}_coxa_servo" type="fixed">
+      <origin rpy="0 0 ${yaw}" xyz="${x} ${y} 0"/>
+      <parent link="${robot_name}/base_center_link"/>
+      <child link="${robot_name}/${prefix}_coxa_servo"/>
+    </joint>
+    <link name="${robot_name}/${prefix}_coxa_servo">
+      <visual>
+        <origin xyz="0 0 0" rpy="0 0 ${-pi/2}" />
+        <geometry>
+          <mesh filename="package://drqp_description/meshes/servo.stl" />
+        </geometry>
+        <material name="drqp_black"/>
+      </visual>
+      <!-- TODO: Define later -->
+      <!-- <collision>
+        <origin rpy="0 0 0" xyz="0 0 0"/>
+        <geometry>
+          <mesh filename="package://drqp_description/meshes/servo.stl" />
+        </geometry>
+      </collision>
+      <inertial>
+        <origin rpy="0 0 0" xyz="0.019066 -0.000002 0.006577"/>
+        <mass value="0.02471" />
+        <inertia ixx="0.0000215400" iyy="0.00002657000" izz="0.00002925000" ixy="-0.00000000122" ixz="-0.00000192741" iyz="-0.00000000001" />
+      </inertial> -->
+    </link>
     <joint name="${prefix}_coxa" type="revolute">
       <axis xyz="0 0 1"/>
       <limit effort="3" lower="${radians(-55)}" upper="${radians(55)}" velocity="${pi}"/>
-      <origin rpy="0 0 ${yaw}" xyz="${x} ${y} 0"/>
-      <parent link="${robot_name}/base_center_link"/>
+      <parent link="${robot_name}/${prefix}_coxa_servo"/>
       <child link="${robot_name}/${prefix}_coxa_link"/>
       <dynamics friction="0.5"/>
@@ -134,7 +159,8 @@
     <link name="${robot_name}/${prefix}_foot_link"/> -->
   </xacro:macro>
+  <xacro:property name="body_height" value="0.037" />
   <link name="$(arg robot_name)/base_center_link">
     <visual>
-      <origin xyz="0 0 0" rpy="${pi/2} 0 ${pi}" />
+      <origin xyz="0 0 -${body_height/2}" rpy="${pi/2} 0 ${pi}" />
       <geometry>
         <mesh filename="package://drqp_description/meshes/body-simple.stl" />
@@ -157,5 +183,5 @@
   </link>
   <joint name="base_bottom" type="fixed">
-    <origin rpy="0 0 0" xyz="0 0 0.033"/>
+    <origin rpy="0 0 0" xyz="0 0 ${body_height/2}"/>
     <child link="$(arg robot_name)/base_center_link"/>
     <parent link="$(arg robot_name)/base_bottom_link"/>

Commit message: Add coxa's two F2 links

File: src/drqp_description/urdf/dr_qp.urdf.xacro (robot description, xacro)
@@ -45,5 +45,5 @@
       <limit effort="3" lower="${radians(-55)}" upper="${radians(55)}" velocity="${pi}"/>
       <parent link="${robot_name}/${prefix}_coxa_servo"/>
-      <child link="${robot_name}/${prefix}_coxa_link"/>
+      <child link="${robot_name}/${prefix}_coxa_f2_link_1"/>
       <dynamics friction="0.5"/>
     </joint>
@@ -57,30 +57,58 @@
       </actuator>
     </transmission>
-    <link name="${robot_name}/${prefix}_coxa_link">
-      <visual>
-        <origin rpy="0 0 0" xyz="0 0 0"/>
-        <geometry>
-          <mesh filename="package://drqp_description/meshes/coxa_link.stl" />
+    <link name="${robot_name}/${prefix}_coxa_f2_link_1">
+      <visual>
+        <origin rpy="0 0 ${pi/2}" xyz="0 0 0"/>
+        <geometry>
+          <mesh filename="package://drqp_description/meshes/F2.stl" />
         </geometry>
         <material name="drqp_black"/>
       </visual>
       <collision>
-        <origin rpy="0 0 0" xyz="0 0 0"/>
-        <geometry>
-          <mesh filename="package://drqp_description/meshes/coxa_link.stl" />
-        </geometry>
-      </collision>
+        <origin rpy="0 0 ${pi/2}" xyz="0 0 0"/>
+        <geometry>
+          <mesh filename="package://drqp_description/meshes/F2.stl" />
+        </geometry>
+      </collision>
+      <!-- TODO: Define later -->
+      <!--
       <inertial>
         <origin rpy="0 0 0" xyz="0.019066 -0.000002 0.006577"/>
         <mass value="0.02471" />
         <inertia ixx="0.0000215400" iyy="0.00002657000" izz="0.00002925000" ixy="-0.00000000122" ixz="-0.00000192741" iyz="-0.00000000001" />
-      </inertial>
-    </link>
-<!--
+      </inertial> -->
+    </link>
+    <joint name="${prefix}_coxa_inner" type="fixed">
+      <origin rpy="${pi/2} 0 0" xyz="${0.0265 * 2} 0 0"/>
+      <parent link="${robot_name}/${prefix}_coxa_f2_link_1"/>
+      <child link="${robot_name}/${prefix}_coxa_f2_link_2"/>
+    </joint>
+    <link name="${robot_name}/${prefix}_coxa_f2_link_2">
+      <visual>
+        <origin rpy="0 0 ${-pi/2}" xyz="0 0 0"/>
+        <geometry>
+          <mesh filename="package://drqp_description/meshes/F2.stl" />
+        </geometry>
+        <material name="drqp_black"/>
+      </visual>
+      <collision>
+        <origin rpy="0 0 ${-pi/2}" xyz="0 0 0"/>
+        <geometry>
+          <mesh filename="package://drqp_description/meshes/F2.stl" />
+        </geometry>
+      </collision>
+      <!-- TODO: Define later -->
+      <!--
+      <inertial>
+        <origin rpy="0 0 0" xyz="0.019066 -0.000002 0.006577"/>
+        <mass value="0.02471" />
+        <inertia ixx="0.0000215400" iyy="0.00002657000" izz="0.00002925000" ixy="-0.00000000122" ixz="-0.00000192741" iyz="-0.00000000001" />
+      </inertial> -->
+    </link>
     <joint name="${prefix}_femur" type="revolute">
       <axis xyz="0 1 0"/>
       <limit effort="3" lower="${radians(-98)}" upper="${radians(90)}" velocity="${pi}"/>
       <origin rpy="0 0 0" xyz="0.052907539 0 0"/>
-      <parent link="${robot_name}/${prefix}_coxa_link"/>
+      <parent link="${robot_name}/${prefix}_coxa_f2_link_2"/>
       <child link="${robot_name}/${prefix}_femur_link"/>
       <dynamics friction="0.5"/>
@@ -103,5 +131,6 @@
         <material name="drqp_black"/>
       </visual>
-      <collision>
+      <!-- TODO: Define later -->
+      <!-- <collision>
         <origin rpy="0 0 0" xyz="0 0 0"/>
         <geometry>
@@ -113,6 +142,7 @@
         <mass value="0.085834" />
         <inertia ixx="0.0000288700" iyy="0.0000750200" izz="0.0000867200" ixy="0.0000002419" ixz="0.0000048494" iyz="0.0000000003" />
-      </inertial>
-    </link>
+      </inertial> -->
+    </link>
+<!--
     <joint name="${prefix}_tibia" type="revolute">
       <axis xyz="0 1 0"/>

Commit message: adjust femur joint position and axis

File: src/drqp_description/urdf/dr_qp.urdf.xacro (robot description, xacro)
@@ -107,7 +107,7 @@
     </link>
     <joint name="${prefix}_femur" type="revolute">
-      <axis xyz="0 1 0"/>
+      <axis xyz="0 0 1"/>
       <limit effort="3" lower="${radians(-98)}" upper="${radians(90)}" velocity="${pi}"/>
-      <origin rpy="0 0 0" xyz="0.052907539 0 0"/>
+      <origin rpy="0 0 0" xyz="0 0 0"/>
       <parent link="${robot_name}/${prefix}_coxa_f2_link_2"/>
       <child link="${robot_name}/${prefix}_femur_link"/>

Commit message: adjust angle limits to the dr.qp model

File: src/drqp_description/urdf/dr_qp.urdf.xacro (robot description, xacro)
@@ -43,5 +43,5 @@
     <joint name="${prefix}_coxa" type="revolute">
       <axis xyz="0 0 1"/>
-      <limit effort="3" lower="${radians(-55)}" upper="${radians(55)}" velocity="${pi}"/>
+      <limit effort="3" lower="${radians(-90)}" upper="${radians(90)}" velocity="${pi}"/>
       <parent link="${robot_name}/${prefix}_coxa_servo"/>
       <child link="${robot_name}/${prefix}_coxa_f2_link_1"/>
@@ -111,5 +111,5 @@
       <origin rpy="0 0 0" xyz="0 0 0"/>
       <parent link="${robot_name}/${prefix}_coxa_f2_link_2"/>
-      <child link="${robot_name}/${prefix}_femur_link"/>
+      <child link="${robot_name}/${prefix}_femur_servo"/>
       <dynamics friction="0.5"/>
     </joint>
@@ -123,4 +123,30 @@
       </actuator>
     </transmission>
+    <link name="${robot_name}/${prefix}_femur_servo">
+      <visual>
+        <origin xyz="0 0 0" rpy="0 0 ${pi/2}" />
+        <geometry>
+          <mesh filename="package://drqp_description/meshes/servo.stl" />
+        </geometry>
+        <material name="drqp_black"/>
+      </visual>
+      <!-- TODO: Define later -->
+      <!-- <collision>
+        <origin rpy="0 0 0" xyz="0 0 0"/>
+        <geometry>
+          <mesh filename="package://drqp_description/meshes/servo.stl" />
+        </geometry>
+      </collision>
+      <inertial>
+        <origin rpy="0 0 0" xyz="0.019066 -0.000002 0.006577"/>
+        <mass value="0.02471" />
+        <inertia ixx="0.0000215400" iyy="0.00002657000" izz="0.00002925000" ixy="-0.00000000122" ixz="-0.00000192741" iyz="-0.00000000001" />
+      </inertial> -->
+    </link>
+    <joint name="${prefix}_femurinner" type="fixed">
+      <origin rpy="0 0 0" xyz="0 0 0"/>
+      <parent link="${robot_name}/${prefix}_femur_servo"/>
+      <child link="${robot_name}/${prefix}_femur_link"/>
+    </joint>
     <link name="${robot_name}/${prefix}_femur_link">
       <visual>

Commit message: add f3 to the model

File: src/drqp_description/urdf/dr_qp.urdf.xacro (robot description, xacro)
@@ -127,4 +127,8 @@
         <origin xyz="0 0 0" rpy="0 0 ${pi/2}" />
         <geometry>
+          <!--
+            Origin is at the actuator center
+            36mm - distance from actuator center to the center of the holes on the back
+           -->
           <mesh filename="package://drqp_description/meshes/servo.stl" />
         </geometry>
@@ -145,23 +149,28 @@
     </link>
     <joint name="${prefix}_femurinner" type="fixed">
-      <origin rpy="0 0 0" xyz="0 0 0"/>
+      <origin rpy="0 0 0" xyz="${0.036 + 0.0055} 0 0"/>
       <parent link="${robot_name}/${prefix}_femur_servo"/>
-      <child link="${robot_name}/${prefix}_femur_link"/>
-    </joint>
-    <link name="${robot_name}/${prefix}_femur_link">
-      <visual>
-        <origin rpy="0 0 0" xyz="0 0 0"/>
-        <geometry>
-          <mesh filename="package://drqp_description/meshes/femur_link.stl" />
-        </geometry>
-        <material name="drqp_black"/>
-      </visual>
-      <!-- TODO: Define later -->
-      <!-- <collision>
-        <origin rpy="0 0 0" xyz="0 0 0"/>
-        <geometry>
-          <mesh filename="package://drqp_description/meshes/femur_link.stl" />
-        </geometry>
-      </collision>
+      <child link="${robot_name}/${prefix}_femur_link_f3"/>
+    </joint>
+    <link name="${robot_name}/${prefix}_femur_link_f3">
+      <visual>
+        <origin rpy="0 0 ${pi/2}" xyz="0 0 0"/>
+        <geometry>
+          <!--
+            Origin is at the center of the flat plane
+            5.5mm - distance from origin to center of the side mounting holes
+           -->
+          <mesh filename="package://drqp_description/meshes/F3.stl" />
+        </geometry>
+        <material name="drqp_black"/>
+      </visual>
+      <collision>
+        <origin rpy="0 0 ${pi/2}" xyz="0 0 0"/>
+        <geometry>
+          <mesh filename="package://drqp_description/meshes/F3.stl" />
+        </geometry>
+      </collision>
+      <!-- TODO: Define later -->
+      <!--
       <inertial>
         <origin rpy="0 0 0" xyz="0.020226 -0.00029 -0.00063"/>

Commit message: affix f1 of femur

File: src/drqp_description/urdf/dr_qp.urdf.xacro (robot description, xacro)
@@ -148,5 +148,5 @@
       </inertial> -->
     </link>
-    <joint name="${prefix}_femurinner" type="fixed">
+    <joint name="${prefix}_femur_inner_1" type="fixed">
       <origin rpy="0 0 0" xyz="${0.036 + 0.0055} 0 0"/>
       <parent link="${robot_name}/${prefix}_femur_servo"/>
@@ -169,4 +169,36 @@
         <geometry>
           <mesh filename="package://drqp_description/meshes/F3.stl" />
+        </geometry>
+      </collision>
+      <!-- TODO: Define later -->
+      <!--
+      <inertial>
+        <origin rpy="0 0 0" xyz="0.020226 -0.00029 -0.00063"/>
+        <mass value="0.085834" />
+        <inertia ixx="0.0000288700" iyy="0.0000750200" izz="0.0000867200" ixy="0.0000002419" ixz="0.0000048494" iyz="0.0000000003" />
+      </inertial> -->
+    </link>
+    <joint name="${prefix}_femur_inner_2" type="fixed">
+      <origin rpy="0 0 0" xyz="0.023 -0.015 0"/>
+      <parent link="${robot_name}/${prefix}_femur_link_f3"/>
+      <child link="${robot_name}/${prefix}_femur_link_f1"/>
+    </joint>
+    <link name="${robot_name}/${prefix}_femur_link_f1">
+      <visual>
+        <origin rpy="${pi} 0 ${pi/2}" xyz="0 0 0"/>
+        <geometry>
+          <!--
+            Origin is at the servo mount/pivot
+            15.0mm - distance from origin to the center mount holes on the mount plane - x axis
+            23.0mm - distance from origin to mount plane - y axis
+           -->
+          <mesh filename="package://drqp_description/meshes/F1.stl" />
+        </geometry>
+        <material name="drqp_black"/>
+      </visual>
+      <collision>
+        <origin rpy="{pi} 0 ${pi/2}" xyz="0 0 0"/>
+        <geometry>
+          <mesh filename="package://drqp_description/meshes/F1.stl" />
         </geometry>
       </collision>

Commit message: fix missing $

File: src/drqp_description/urdf/dr_qp.urdf.xacro (robot description, xacro)
@@ -198,5 +198,5 @@
       </visual>
       <collision>
-        <origin rpy="{pi} 0 ${pi/2}" xyz="0 0 0"/>
+        <origin rpy="${pi} 0 ${pi/2}" xyz="0 0 0"/>
         <geometry>
           <mesh filename="package://drqp_description/meshes/F1.stl" />
