Commit message: add tibia servo

File: src/drqp_description/urdf/dr_qp.urdf.xacro (robot description, xacro)
@@ -211,11 +211,10 @@
       </inertial> -->
     </link>
-<!--
     <joint name="${prefix}_tibia" type="revolute">
-      <axis xyz="0 1 0"/>
-      <limit effort="3" lower="${radians(-45)}" upper="${radians(125)}" velocity="${pi}"/>
-      <origin rpy="0 0 0" xyz="0.06 0 -0.015"/>
-      <parent link="${robot_name}/${prefix}_femur_link"/>
-      <child link="${robot_name}/${prefix}_tibia_link"/>
+      <axis xyz="0 0 1"/>
+      <limit effort="3" lower="${radians(-125)}" upper="${radians(80)}" velocity="${pi}"/>
+      <origin rpy="0 0 0" xyz="0 0 0"/>
+      <parent link="${robot_name}/${prefix}_femur_link_f1"/>
+      <child link="${robot_name}/${prefix}_tibia_servo"/>
       <dynamics friction="0.5"/>
     </joint>
@@ -229,16 +228,18 @@
       </actuator>
     </transmission>
-    <link name="${robot_name}/${prefix}_tibia_link">
-      <visual>
-        <origin rpy="0 0 0" xyz="0 0 0"/>
-        <geometry>
-          <mesh filename="package://drqp_description/meshes/tibia_link.stl" />
-        </geometry>
-        <material name="drqp_black"/>
-      </visual>
-      <collision>
-        <origin rpy="0 0 0" xyz="0 0 0"/>
-        <geometry>
-          <mesh filename="package://drqp_description/meshes/tibia_link.stl" />
+    <link name="${robot_name}/${prefix}_tibia_servo">
+      <visual>
+        <origin xyz="0 0 0" rpy="0 0 ${pi/2}" />
+        <geometry>
+          <mesh filename="package://drqp_description/meshes/servo.stl" />
+        </geometry>
+        <material name="drqp_black"/>
+      </visual>
+      <!-- TODO: Define later -->
+      <!--
+      <collision>
+        <origin xyz="0 0 0" rpy="0 0 ${pi/2}" />
+        <geometry>
+          <mesh filename="package://drqp_description/meshes/servo.stl" />
         </geometry>
       </collision>
@@ -248,8 +249,10 @@
         <inertia ixx="0.0001762000" iyy="0.0005158000" izz="0.0003768000" ixy="-0.0000014522" ixz="0.0001789000" iyz="0.0000006181" />
       </inertial>
-    </link>
+      -->
+    </link>
+<!--
     <joint name="${prefix}_foot" type="fixed">
       <origin rpy="0 0 0" xyz="0.095 0 -0.09"/>
-      <parent link="${robot_name}/${prefix}_tibia_link"/>
+      <parent link="${robot_name}/${prefix}_tibia_servo"/>
       <child link="${robot_name}/${prefix}_foot_link"/>
     </joint>

Commit message: fix all links to be z up visual up to femur

File: src/drqp_description/urdf/dr_qp.urdf.xacro (robot description, xacro)
@@ -80,5 +80,5 @@
     </link>
     <joint name="${prefix}_coxa_inner" type="fixed">
-      <origin rpy="${pi/2} 0 0" xyz="${0.0265 * 2} 0 0"/>
+      <origin rpy="0 0 0" xyz="${0.0265 * 2} 0 0"/>
       <parent link="${robot_name}/${prefix}_coxa_f2_link_1"/>
       <child link="${robot_name}/${prefix}_coxa_f2_link_2"/>
@@ -86,5 +86,5 @@
     <link name="${robot_name}/${prefix}_coxa_f2_link_2">
       <visual>
-        <origin rpy="0 0 ${-pi/2}" xyz="0 0 0"/>
+        <origin rpy="0 ${pi/2} ${-pi/2}" xyz="0 0 0"/>
         <geometry>
           <mesh filename="package://drqp_description/meshes/F2.stl" />
@@ -93,5 +93,5 @@
       </visual>
       <collision>
-        <origin rpy="0 0 ${-pi/2}" xyz="0 0 0"/>
+        <origin rpy="0 ${pi/2} ${-pi/2}" xyz="0 0 0"/>
         <geometry>
           <mesh filename="package://drqp_description/meshes/F2.stl" />
@@ -107,5 +107,5 @@
     </link>
     <joint name="${prefix}_femur" type="revolute">
-      <axis xyz="0 0 1"/>
+      <axis xyz="0 1 0"/>
       <limit effort="3" lower="${radians(-98)}" upper="${radians(90)}" velocity="${pi}"/>
       <origin rpy="0 0 0" xyz="0 0 0"/>
@@ -125,5 +125,5 @@
     <link name="${robot_name}/${prefix}_femur_servo">
       <visual>
-        <origin xyz="0 0 0" rpy="0 0 ${pi/2}" />
+        <origin rpy="0 ${pi/2} ${pi/2}" xyz="0 0 0" />
         <geometry>
           <!--
@@ -212,5 +212,5 @@
     </link>
     <joint name="${prefix}_tibia" type="revolute">
-      <axis xyz="0 0 1"/>
+      <axis xyz="0 1 0"/>
       <limit effort="3" lower="${radians(-125)}" upper="${radians(80)}" velocity="${pi}"/>
       <origin rpy="0 0 0" xyz="0 0 0"/>
@@ -250,4 +250,34 @@
       </inertial>
       -->
+    </link>
+    <joint name="${prefix}_tibia_leg" type="fixed">
+      <origin rpy="0 0 0" xyz="0.0325 0 0"/>
+      <parent link="${robot_name}/${prefix}_tibia_servo"/>
+      <child link="${robot_name}/${prefix}_tibia_leg"/>
+    </joint>
+    <link name="${robot_name}/${prefix}_tibia_leg">
+      <visual>
+        <origin rpy="0 0 0" xyz="0 0 0"/>
+        <geometry>
+          <!--
+            Origin is at end servo attachment, 32.5 between servo pivot and this point
+           -->
+          <mesh filename="package://drqp_description/meshes/Tibia.stl" />
+        </geometry>
+        <material name="drqp_black"/>
+      </visual>
+      <collision>
+        <origin rpy="0 0 0" xyz="0 0 0"/>
+        <geometry>
+          <mesh filename="package://drqp_description/meshes/Tibia.stl" />
+        </geometry>
+      </collision>
+      <!-- TODO: Define later -->
+      <!--
+      <inertial>
+        <origin rpy="0 0 0" xyz="0.020226 -0.00029 -0.00063"/>
+        <mass value="0.085834" />
+        <inertia ixx="0.0000288700" iyy="0.0000750200" izz="0.0000867200" ixy="0.0000002419" ixz="0.0000048494" iyz="0.0000000003" />
+      </inertial> -->
     </link>
 <!--
@@ -288,9 +318,9 @@
   </joint>
   <xacro:leg robot_name="$(arg robot_name)" prefix="right_front" x="0.11692" y="-0.06387" yaw="${-pi/4}"/>
-  <xacro:leg robot_name="$(arg robot_name)" prefix="right_middle" x="0" y="-0.103" yaw="${-pi/2}"/>
+  <!-- <xacro:leg robot_name="$(arg robot_name)" prefix="right_middle" x="0" y="-0.103" yaw="${-pi/2}"/>
   <xacro:leg robot_name="$(arg robot_name)" prefix="right_back" x="-0.11692" y="-0.06387" yaw="${-3*pi/4}"/>
   <xacro:leg robot_name="$(arg robot_name)" prefix="left_front" x="0.11692" y="0.06387" yaw="${pi/4}"/>
   <xacro:leg robot_name="$(arg robot_name)" prefix="left_middle" x="0" y="0.103" yaw="${pi/2}"/>
-  <xacro:leg robot_name="$(arg robot_name)" prefix="left_back" x="-0.11692" y="0.06387" yaw="${3*pi/4}"/>
+  <xacro:leg robot_name="$(arg robot_name)" prefix="left_back" x="-0.11692" y="0.06387" yaw="${3*pi/4}"/> -->
   <xacro:if value="${urdf_loc != ''}">
     <xacro:include filename="${urdf_loc}"/>

Commit message: femur aligned

File: src/drqp_description/urdf/dr_qp.urdf.xacro (robot description, xacro)
@@ -155,5 +155,5 @@
     <link name="${robot_name}/${prefix}_femur_link_f3">
       <visual>
-        <origin rpy="0 0 ${pi/2}" xyz="0 0 0"/>
+        <origin rpy="0 ${pi/2} ${pi/2}" xyz="0 0 0"/>
         <geometry>
           <!--
@@ -166,5 +166,5 @@
       </visual>
       <collision>
-        <origin rpy="0 0 ${pi/2}" xyz="0 0 0"/>
+        <origin rpy="0 ${pi/2} ${pi/2}" xyz="0 0 0"/>
         <geometry>
           <mesh filename="package://drqp_description/meshes/F3.stl" />
@@ -180,5 +180,5 @@
     </link>
     <joint name="${prefix}_femur_inner_2" type="fixed">
-      <origin rpy="0 0 0" xyz="0.023 -0.015 0"/>
+      <origin rpy="0 0 0" xyz="0.023 0 -0.015"/>
       <parent link="${robot_name}/${prefix}_femur_link_f3"/>
       <child link="${robot_name}/${prefix}_femur_link_f1"/>
@@ -186,5 +186,5 @@
     <link name="${robot_name}/${prefix}_femur_link_f1">
       <visual>
-        <origin rpy="${pi} 0 ${pi/2}" xyz="0 0 0"/>
+        <origin rpy="${pi} ${-pi/2} ${pi/2}" xyz="0 0 0"/>
         <geometry>
           <!--
@@ -198,5 +198,5 @@
       </visual>
       <collision>
-        <origin rpy="${pi} 0 ${pi/2}" xyz="0 0 0"/>
+        <origin rpy="${pi} ${-pi/2} ${pi/2}" xyz="0 0 0"/>
         <geometry>
           <mesh filename="package://drqp_description/meshes/F1.stl" />

Commit message: all aligned tibia stl is origin is way off

File: src/drqp_description/urdf/dr_qp.urdf.xacro (robot description, xacro)
@@ -230,14 +230,14 @@
     <link name="${robot_name}/${prefix}_tibia_servo">
       <visual>
-        <origin xyz="0 0 0" rpy="0 0 ${pi/2}" />
-        <geometry>
-          <mesh filename="package://drqp_description/meshes/servo.stl" />
-        </geometry>
-        <material name="drqp_black"/>
-      </visual>
-      <!-- TODO: Define later -->
-      <!--
-      <collision>
-        <origin xyz="0 0 0" rpy="0 0 ${pi/2}" />
+        <origin rpy="0 ${pi/2} ${pi/2}" xyz="0 0 0" />
+        <geometry>
+          <mesh filename="package://drqp_description/meshes/servo.stl" />
+        </geometry>
+        <material name="drqp_black"/>
+      </visual>
+      <!-- TODO: Define later -->
+      <!--
+      <collision>
+        <origin rpy="0 ${pi/2} ${pi/2}" xyz="0 0 0"" />
         <geometry>
           <mesh filename="package://drqp_description/meshes/servo.stl" />

Commit message: define foot

File: src/drqp_description/urdf/dr_qp.urdf.xacro (robot description, xacro)
@@ -281,11 +281,10 @@
       </inertial> -->
     </link>
-<!--
     <joint name="${prefix}_foot" type="fixed">
-      <origin rpy="0 0 0" xyz="0.095 0 -0.09"/>
-      <parent link="${robot_name}/${prefix}_tibia_servo"/>
+      <origin rpy="0 0 0" xyz="0.052797 0 -0.088395"/>
+      <parent link="${robot_name}/${prefix}_tibia_leg"/>
       <child link="${robot_name}/${prefix}_foot_link"/>
     </joint>
-    <link name="${robot_name}/${prefix}_foot_link"/> -->
+    <link name="${robot_name}/${prefix}_foot_link"/>
   </xacro:macro>
   <xacro:property name="body_height" value="0.037" />

Commit message: add joint for camera

File: src/drqp_description/urdf/dr_qp.urdf.xacro (robot description, xacro)
@@ -313,7 +313,14 @@
   <joint name="base_bottom" type="fixed">
     <origin rpy="0 0 0" xyz="0 0 ${body_height/2}"/>
+    <parent link="$(arg robot_name)/base_bottom_link"/>
     <child link="$(arg robot_name)/base_center_link"/>
+  </joint>
+  <joint name="base_bottom_to_camera" type="fixed">
+    <origin rpy="0 0 0" xyz="0.132 0 0.019"/>
     <parent link="$(arg robot_name)/base_bottom_link"/>
+    <child link="$(arg robot_name)/camera"/>
   </joint>
+  <link name="$(arg robot_name)/camera">
+  </link>
   <xacro:leg robot_name="$(arg robot_name)" prefix="right_front" x="0.11692" y="-0.06387" yaw="${-pi/4}"/>
   <xacro:leg robot_name="$(arg robot_name)" prefix="right_middle" x="0" y="-0.103" yaw="${-pi/2}"/>

Commit message: use center link as parent for acemra

File: src/drqp_description/urdf/dr_qp.urdf.xacro (robot description, xacro)
@@ -317,6 +317,6 @@
   </joint>
   <joint name="base_bottom_to_camera" type="fixed">
-    <origin rpy="0 0 0" xyz="0.132 0 0.019"/>
-    <parent link="$(arg robot_name)/base_bottom_link"/>
+    <origin rpy="0 0 0" xyz="0.132 0 0"/>
+    <parent link="$(arg robot_name)/base_center_link"/>
     <child link="$(arg robot_name)/camera"/>
   </joint>

Commit message: base_bottom_link is world for this single robot

File: src/drqp_description/urdf/dr_qp.urdf.xacro (robot description, xacro)
@@ -309,5 +309,5 @@
     </inertial>
   </link>
-  <link name="$(arg robot_name)/base_bottom_link">
+  <link name="$(arg robot_name)/base_bottom_link"> <!-- AKA World -->
   </link>
   <joint name="base_bottom" type="fixed">

Commit message: rename base_link

File: src/drqp_description/urdf/dr_qp.urdf.xacro (robot description, xacro)
@@ -309,9 +309,9 @@
     </inertial>
   </link>
-  <link name="$(arg robot_name)/base_bottom_link"> <!-- AKA World -->
+  <link name="$(arg robot_name)/base_link"> <!-- AKA World -->
   </link>
   <joint name="base_bottom" type="fixed">
     <origin rpy="0 0 0" xyz="0 0 ${body_height/2}"/>
-    <parent link="$(arg robot_name)/base_bottom_link"/>
+    <parent link="$(arg robot_name)/base_link"/>
     <child link="$(arg robot_name)/base_center_link"/>
   </joint>
