Commit message: split into couple xacro files

File: src/drqp_description/urdf/dr_qp.urdf.xacro (robot description, xacro)
@@ -14,313 +14,6 @@
     <color rgba="0.5 0.5 0.5 0.2" />
   </material>
-  <xacro:macro name="leg" params="robot_name prefix x y yaw">
-    <joint name="${prefix}_coxa_servo" type="fixed">
-      <origin rpy="0 0 ${yaw}" xyz="${x} ${y} 0"/>
-      <parent link="${robot_name}/base_center_link"/>
-      <child link="${robot_name}/${prefix}_coxa_servo"/>
-    </joint>
-    <link name="${robot_name}/${prefix}_coxa_servo">
-      <visual>
-        <origin xyz="0 0 0" rpy="0 0 ${-pi/2}" />
-        <geometry>
-          <mesh filename="package://drqp_description/meshes/servo.stl" />
-        </geometry>
-        <material name="drqp_black"/>
-      </visual>
-      <!-- TODO: Define later -->
-      <!-- <collision>
-        <origin rpy="0 0 0" xyz="0 0 0"/>
-        <geometry>
-          <mesh filename="package://drqp_description/meshes/servo.stl" />
-        </geometry>
-      </collision>
-      <inertial>
-        <origin rpy="0 0 0" xyz="0.019066 -0.000002 0.006577"/>
-        <mass value="0.02471" />
-        <inertia ixx="0.0000215400" iyy="0.00002657000" izz="0.00002925000" ixy="-0.00000000122" ixz="-0.00000192741" iyz="-0.00000000001" />
-      </inertial> -->
-    </link>
-    <joint name="${prefix}_coxa" type="revolute">
-      <axis xyz="0 0 1"/>
-      <limit effort="3" lower="${radians(-90)}" upper="${radians(90)}" velocity="${pi}"/>
-      <parent link="${robot_name}/${prefix}_coxa_servo"/>
-      <child link="${robot_name}/${prefix}_coxa_f2_link_1"/>
-      <dynamics friction="0.5"/>
-    </joint>
-    <transmission name="trans_${prefix}_coxa">
-      <type>transmission_interface/SimpleTransmission</type>
-      <joint name="${prefix}_coxa">
-        <hardwareInterface>hardware_interface/EffortJointInterface</hardwareInterface>
-      </joint>
-      <actuator name="${prefix}_coxa_motor">
-        <mechanicalReduction>1</mechanicalReduction>
-      </actuator>
-    </transmission>
-    <link name="${robot_name}/${prefix}_coxa_f2_link_1">
-      <visual>
-        <origin rpy="0 0 ${pi/2}" xyz="0 0 0"/>
-        <geometry>
-          <mesh filename="package://drqp_description/meshes/F2.stl" />
-        </geometry>
-        <material name="drqp_black"/>
-      </visual>
-      <collision>
-        <origin rpy="0 0 ${pi/2}" xyz="0 0 0"/>
-        <geometry>
-          <mesh filename="package://drqp_description/meshes/F2.stl" />
-        </geometry>
-      </collision>
-      <!-- TODO: Define later -->
-      <!--
-      <inertial>
-        <origin rpy="0 0 0" xyz="0.019066 -0.000002 0.006577"/>
-        <mass value="0.02471" />
-        <inertia ixx="0.0000215400" iyy="0.00002657000" izz="0.00002925000" ixy="-0.00000000122" ixz="-0.00000192741" iyz="-0.00000000001" />
-      </inertial> -->
-    </link>
-    <joint name="${prefix}_coxa_inner" type="fixed">
-      <origin rpy="0 0 0" xyz="${0.0265 * 2} 0 0"/>
-      <parent link="${robot_name}/${prefix}_coxa_f2_link_1"/>
-      <child link="${robot_name}/${prefix}_coxa_f2_link_2"/>
-    </joint>
-    <link name="${robot_name}/${prefix}_coxa_f2_link_2">
-      <visual>
-        <origin rpy="0 ${pi/2} ${-pi/2}" xyz="0 0 0"/>
-        <geometry>
-          <mesh filename="package://drqp_description/meshes/F2.stl" />
-        </geometry>
-        <material name="drqp_black"/>
-      </visual>
-      <collision>
-        <origin rpy="0 ${pi/2} ${-pi/2}" xyz="0 0 0"/>
-        <geometry>
-          <mesh filename="package://drqp_description/meshes/F2.stl" />
-        </geometry>
-      </collision>
-      <!-- TODO: Define later -->
-      <!--
-      <inertial>
-        <origin rpy="0 0 0" xyz="0.019066 -0.000002 0.006577"/>
-        <mass value="0.02471" />
-        <inertia ixx="0.0000215400" iyy="0.00002657000" izz="0.00002925000" ixy="-0.00000000122" ixz="-0.00000192741" iyz="-0.00000000001" />
-      </inertial> -->
-    </link>
-    <joint name="${prefix}_femur" type="revolute">
-      <axis xyz="0 1 0"/>
-      <limit effort="3" lower="${radians(-98)}" upper="${radians(90)}" velocity="${pi}"/>
-      <origin rpy="0 0 0" xyz="0 0 0"/>
-      <parent link="${robot_name}/${prefix}_coxa_f2_link_2"/>
-      <child link="${robot_name}/${prefix}_femur_servo"/>
-      <dynamics friction="0.5"/>
-    </joint>
-    <transmission name="trans_${prefix}_femur">
-      <type>transmission_interface/SimpleTransmission</type>
-      <joint name="${prefix}_femur">
-        <hardwareInterface>hardware_interface/EffortJointInterface</hardwareInterface>
-      </joint>
-      <actuator name="${prefix}_femur_motor">
-        <mechanicalReduction>1</mechanicalReduction>
-      </actuator>
-    </transmission>
-    <link name="${robot_name}/${prefix}_femur_servo">
-      <visual>
-        <origin rpy="0 ${pi/2} ${pi/2}" xyz="0 0 0" />
-        <geometry>
-          <!--
-            Origin is at the actuator center
-            36mm - distance from actuator center to the center of the holes on the back
-           -->
-          <mesh filename="package://drqp_description/meshes/servo.stl" />
-        </geometry>
-        <material name="drqp_black"/>
-      </visual>
-      <!-- TODO: Define later -->
-      <!-- <collision>
-        <origin rpy="0 0 0" xyz="0 0 0"/>
-        <geometry>
-          <mesh filename="package://drqp_description/meshes/servo.stl" />
-        </geometry>
-      </collision>
-      <inertial>
-        <origin rpy="0 0 0" xyz="0.019066 -0.000002 0.006577"/>
-        <mass value="0.02471" />
-        <inertia ixx="0.0000215400" iyy="0.00002657000" izz="0.00002925000" ixy="-0.00000000122" ixz="-0.00000192741" iyz="-0.00000000001" />
-      </inertial> -->
-    </link>
-    <joint name="${prefix}_femur_inner_1" type="fixed">
-      <origin rpy="0 0 0" xyz="${0.036 + 0.0055} 0 0"/>
-      <parent link="${robot_name}/${prefix}_femur_servo"/>
-      <child link="${robot_name}/${prefix}_femur_link_f3"/>
-    </joint>
-    <link name="${robot_name}/${prefix}_femur_link_f3">
-      <visual>
-        <origin rpy="0 ${pi/2} ${pi/2}" xyz="0 0 0"/>
-        <geometry>
-          <!--
-            Origin is at the center of the flat plane
-            5.5mm - distance from origin to center of the side mounting holes
-           -->
-          <mesh filename="package://drqp_description/meshes/F3.stl" />
-        </geometry>
-        <material name="drqp_black"/>
-      </visual>
-      <collision>
-        <origin rpy="0 ${pi/2} ${pi/2}" xyz="0 0 0"/>
-        <geometry>
-          <mesh filename="package://drqp_description/meshes/F3.stl" />
-        </geometry>
-      </collision>
-      <!-- TODO: Define later -->
-      <!--
-      <inertial>
-        <origin rpy="0 0 0" xyz="0.020226 -0.00029 -0.00063"/>
-        <mass value="0.085834" />
-        <inertia ixx="0.0000288700" iyy="0.0000750200" izz="0.0000867200" ixy="0.0000002419" ixz="0.0000048494" iyz="0.0000000003" />
-      </inertial> -->
-    </link>
-    <joint name="${prefix}_femur_inner_2" type="fixed">
-      <origin rpy="0 0 0" xyz="0.023 0 -0.015"/>
-      <parent link="${robot_name}/${prefix}_femur_link_f3"/>
-      <child link="${robot_name}/${prefix}_femur_link_f1"/>
-    </joint>
-    <link name="${robot_name}/${prefix}_femur_link_f1">
-      <visual>
-        <origin rpy="${pi} ${-pi/2} ${pi/2}" xyz="0 0 0"/>
-        <geometry>
-          <!--
-            Origin is at the servo mount/pivot
-            15.0mm - distance from origin to the center mount holes on the mount plane - x axis
-            23.0mm - distance from origin to mount plane - y axis
-           -->
-          <mesh filename="package://drqp_description/meshes/F1.stl" />
-        </geometry>
-        <material name="drqp_black"/>
-      </visual>
-      <collision>
-        <origin rpy="${pi} ${-pi/2} ${pi/2}" xyz="0 0 0"/>
-        <geometry>
-          <mesh filename="package://drqp_description/meshes/F1.stl" />
-        </geometry>
-      </collision>
-      <!-- TODO: Define later -->
-      <!--
-      <inertial>
-        <origin rpy="0 0 0" xyz="0.020226 -0.00029 -0.00063"/>
-        <mass value="0.085834" />
-        <inertia ixx="0.0000288700" iyy="0.0000750200" izz="0.0000867200" ixy="0.0000002419" ixz="0.0000048494" iyz="0.0000000003" />
-      </inertial> -->
-    </link>
-    <joint name="${prefix}_tibia" type="revolute">
-      <axis xyz="0 1 0"/>
-      <limit effort="3" lower="${radians(-125)}" upper="${radians(80)}" velocity="${pi}"/>
-      <origin rpy="0 0 0" xyz="0 0 0"/>
-      <parent link="${robot_name}/${prefix}_femur_link_f1"/>
-      <child link="${robot_name}/${prefix}_tibia_servo"/>
-      <dynamics friction="0.5"/>
-    </joint>
-    <transmission name="trans_${prefix}_tibia">
-      <type>transmission_interface/SimpleTransmission</type>
-      <joint name="${prefix}_tibia">
-        <hardwareInterface>hardware_interface/EffortJointInterface</hardwareInterface>
-      </joint>
-      <actuator name="${prefix}_tibia_motor">
-        <mechanicalReduction>1</mechanicalReduction>
-      </actuator>
-    </transmission>
-    <link name="${robot_name}/${prefix}_tibia_servo">
-      <visual>
-        <origin rpy="0 ${pi/2} ${pi/2}" xyz="0 0 0" />
-        <geometry>
-          <mesh filename="package://drqp_description/meshes/servo.stl" />
-        </geometry>
-        <material name="drqp_black"/>
-      </visual>
-      <!-- TODO: Define later -->
-      <!--
-      <collision>
-        <origin rpy="0 ${pi/2} ${pi/2}" xyz="0 0 0"" />
-        <geometry>
-          <mesh filename="package://drqp_description/meshes/servo.stl" />
-        </geometry>
-      </collision>
-      <inertial>
-        <origin rpy="0 0 0" xyz="0.036797 0.000054 -0.011991"/>
-        <mass value="0.171825" />
-        <inertia ixx="0.0001762000" iyy="0.0005158000" izz="0.0003768000" ixy="-0.0000014522" ixz="0.0001789000" iyz="0.0000006181" />
-      </inertial>
-      -->
-    </link>
-    <joint name="${prefix}_tibia_leg" type="fixed">
-      <origin rpy="0 0 0" xyz="0.0325 0 0"/>
-      <parent link="${robot_name}/${prefix}_tibia_servo"/>
-      <child link="${robot_name}/${prefix}_tibia_leg"/>
-    </joint>
-    <link name="${robot_name}/${prefix}_tibia_leg">
-      <visual>
-        <origin rpy="0 0 0" xyz="0 0 0"/>
-        <geometry>
-          <!--
-            Origin is at end servo attachment, 32.5 between servo pivot and this point
-           -->
-          <mesh filename="package://drqp_description/meshes/Tibia.stl" />
-        </geometry>
-        <material name="drqp_black"/>
-      </visual>
-      <collision>
-        <origin rpy="0 0 0" xyz="0 0 0"/>
-        <geometry>
-          <mesh filename="package://drqp_description/meshes/Tibia.stl" />
-        </geometry>
-      </collision>
-      <!-- TODO: Define later -->
-      <!--
-      <inertial>
-        <origin rpy="0 0 0" xyz="0.020226 -0.00029 -0.00063"/>
-        <mass value="0.085834" />
-        <inertia ixx="0.0000288700" iyy="0.0000750200" izz="0.0000867200" ixy="0.0000002419" ixz="0.0000048494" iyz="0.0000000003" />
-      </inertial> -->
-    </link>
-    <joint name="${prefix}_foot" type="fixed">
-      <origin rpy="0 0 0" xyz="0.052797 0 -0.088395"/>
-      <parent link="${robot_name}/${prefix}_tibia_leg"/>
-      <child link="${robot_name}/${prefix}_foot_link"/>
-    </joint>
-    <link name="${robot_name}/${prefix}_foot_link"/>
-  </xacro:macro>
-  <xacro:property name="body_height" value="0.037" />
-  <link name="$(arg robot_name)/base_center_link">
-    <visual>
-      <origin xyz="0 0 -${body_height/2}" rpy="${pi/2} 0 ${pi}" />
-      <geometry>
-        <mesh filename="package://drqp_description/meshes/body-simple.stl" />
-      </geometry>
-      <material name="drqp_black"/>
-    </visual>
-    <collision>
-      <origin xyz="0 0 0" rpy="${pi/2} 0 ${pi}" />
-      <geometry>
-        <mesh filename="package://drqp_description/meshes/body-simple.stl" />
-      </geometry>
-    </collision>
-    <inertial>
-      <origin rpy="0 0 0" xyz="0.001522 0.000302 0.015345"/>
-      <mass value="1.522054" />
-      <inertia ixx="0.0044660000" iyy="0.0084890000" izz="0.0092020000" ixy="0.0000076888" ixz="-0.0001245000" iyz="0.0000050996" />
-    </inertial>
-  </link>
-  <link name="$(arg robot_name)/base_link"> <!-- AKA World -->
-  </link>
-  <joint name="base_bottom" type="fixed">
-    <origin rpy="0 0 0" xyz="0 0 ${body_height/2}"/>
-    <parent link="$(arg robot_name)/base_link"/>
-    <child link="$(arg robot_name)/base_center_link"/>
-  </joint>
-  <joint name="base_bottom_to_camera" type="fixed">
-    <origin rpy="0 0 0" xyz="0.132 0 0"/>
-    <parent link="$(arg robot_name)/base_center_link"/>
-    <child link="$(arg robot_name)/camera"/>
-  </joint>
-  <link name="$(arg robot_name)/camera">
-  </link>
+  <xacro:include filename="$(find drqp_description)/urdf/body.urdf.xacro"/>
+  <xacro:include filename="$(find drqp_description)/urdf/leg.urdf.xacro"/>
   <xacro:leg robot_name="$(arg robot_name)" prefix="right_front" x="0.11692" y="-0.06387" yaw="${-pi/4}"/>
   <xacro:leg robot_name="$(arg robot_name)" prefix="right_middle" x="0" y="-0.103" yaw="${-pi/2}"/>
