Commit message: fix collisions origin

File: src/drqp_description/urdf/body.urdf.xacro (robot description, xacro)
@@ -11,5 +11,5 @@
     </visual>
     <collision>
-      <origin xyz="0 0 0" rpy="${pi/2} 0 ${pi}" />
+      <origin xyz="0 0 -${body_height/2}" rpy="${pi/2} 0 ${pi}" />
       <geometry>
         <mesh filename="package://drqp_description/meshes/body-simple.stl" />

Commit message: add collision geoms and use them in urdf

File: src/drqp_description/urdf/body.urdf.xacro (robot description, xacro)
@@ -11,7 +11,7 @@
     </visual>
     <collision>
-      <origin xyz="0 0 -${body_height/2}" rpy="${pi/2} 0 ${pi}" />
+      <origin xyz="0 0 -${body_height/2}" rpy="0 0 0" />
       <geometry>
-        <mesh filename="package://drqp_description/meshes/body-simple.stl" />
+        <mesh filename="package://drqp_description/meshes/body-collision.stl" />
       </geometry>
     </collision>

File: src/drqp_description/urdf/leg.urdf.xacro (robot description, xacro)
@@ -28,5 +28,5 @@
       <origin xyz="0 0 0" rpy="0 0 ${-pi/2}" />
       <geometry>
-        <mesh filename="package://drqp_description/meshes/servo.stl" />
+        <mesh filename="package://drqp_description/meshes/servo-collision.stl" />
       </geometry>
     </collision>
@@ -64,5 +64,5 @@
       <origin rpy="0 0 ${pi/2}" xyz="0 0 0"/>
       <geometry>
-        <mesh filename="package://drqp_description/meshes/F2.stl" />
+        <mesh filename="package://drqp_description/meshes/F2-collision.stl" />
       </geometry>
     </collision>
@@ -88,5 +88,5 @@
       <origin rpy="0 ${pi/2} ${-pi/2}" xyz="0 0 0"/>
       <geometry>
-        <mesh filename="package://drqp_description/meshes/F2.stl" />
+        <mesh filename="package://drqp_description/meshes/F2-collision.stl" />
       </geometry>
     </collision>
@@ -125,5 +125,5 @@
       <origin rpy="0 ${pi/2} ${pi/2}" xyz="0 0 0" />
       <geometry>
-        <mesh filename="package://drqp_description/meshes/servo.stl" />
+        <mesh filename="package://drqp_description/meshes/servo-collision.stl" />
       </geometry>
     </collision>
@@ -157,5 +157,5 @@
       <origin rpy="0 ${pi/2} ${pi/2}" xyz="0 0 0"/>
       <geometry>
-        <mesh filename="package://drqp_description/meshes/F3.stl" />
+        <mesh filename="package://drqp_description/meshes/F3-collision.stl" />
       </geometry>
     </collision>
@@ -186,5 +186,5 @@
       <origin rpy="${pi} ${-pi/2} ${pi/2}" xyz="0 0 0"/>
       <geometry>
-        <mesh filename="package://drqp_description/meshes/F1.stl" />
+        <mesh filename="package://drqp_description/meshes/F1-collision.stl" />
       </geometry>
     </collision>
@@ -219,5 +219,5 @@
       <origin rpy="0 ${pi/2} ${pi/2}" xyz="0 0 0" />
       <geometry>
-        <mesh filename="package://drqp_description/meshes/servo.stl" />
+        <mesh filename="package://drqp_description/meshes/servo-collision.stl" />
       </geometry>
     </collision>
@@ -250,5 +250,5 @@
       <origin rpy="0 0 0" xyz="0 0 0"/>
       <geometry>
-        <mesh filename="package://drqp_description/meshes/Tibia.stl" />
+        <mesh filename="package://drqp_description/meshes/Tibia-collision.stl" />
       </geometry>
     </collision>
