Commit message: switch to position control add publishing of fixed joints

File: src/drqp_description/urdf/gazebo.xacro (robot description, xacro)
@@ -7,12 +7,13 @@
         <xacro:macro name="hexjoint" params="name">
             <joint name="${name}">
-                <command_interface name="effort">
-                    <!-- ros2 topic pub /effort_controllers/commands std_msgs/msg/Float64MultiArray "{data: [20,20,20,20,20,20,20,20,20,20,20,20,20,20,20,20,20,20],layout: {dim:[], data_offset: 1}}" -->
-                    <!-- <param name="min">-1800</param>
-                    <param name="max">1800</param> -->
+                <command_interface name="position">
+                    <param name="min">-15</param>
+                    <param name="max">15</param>
                 </command_interface>
-                <!-- <state_interface name="position"/> -->
+                <state_interface name="position">
+                  <param name="initial_value">0</param>
+                </state_interface>
+                <state_interface name="velocity"/>
                 <state_interface name="effort"/>
-                <!-- <state_interface name="current"/> -->
             </joint>
         </xacro:macro>

File: src/drqp_description/urdf/leg.urdf.xacro (robot description, xacro)
@@ -47,13 +47,4 @@
     <dampingFactor>0.2</dampingFactor>
   </gazebo>
-  <transmission name="trans_${prefix}_coxa">
-    <type>transmission_interface/SimpleTransmission</type>
-    <joint name="${prefix}_coxa">
-      <hardwareInterface>hardware_interface/EffortJointInterface</hardwareInterface>
-    </joint>
-    <actuator name="${prefix}_coxa_motor">
-      <mechanicalReduction>1</mechanicalReduction>
-    </actuator>
-  </transmission>
   <link name="${robot_name}/${prefix}_coxa_f2_link_1">
     <visual>
@@ -107,13 +98,4 @@
     <dampingFactor>0.2</dampingFactor>
   </gazebo>
-  <transmission name="trans_${prefix}_femur">
-    <type>transmission_interface/SimpleTransmission</type>
-    <joint name="${prefix}_femur">
-      <hardwareInterface>hardware_interface/EffortJointInterface</hardwareInterface>
-    </joint>
-    <actuator name="${prefix}_femur_motor">
-      <mechanicalReduction>1</mechanicalReduction>
-    </actuator>
-  </transmission>
   <link name="${robot_name}/${prefix}_femur_servo">
     <visual>
@@ -208,13 +190,4 @@
     <dampingFactor>0.2</dampingFactor>
   </gazebo>
-  <transmission name="trans_${prefix}_tibia">
-    <type>transmission_interface/SimpleTransmission</type>
-    <joint name="${prefix}_tibia">
-      <hardwareInterface>hardware_interface/EffortJointInterface</hardwareInterface>
-    </joint>
-    <actuator name="${prefix}_tibia_motor">
-      <mechanicalReduction>1</mechanicalReduction>
-    </actuator>
-  </transmission>
   <link name="${robot_name}/${prefix}_tibia_servo">
     <visual>
