Commit message: define collisions same as visual inertial is kinda random

File: src/drqp_description/urdf/leg.urdf.xacro (robot description, xacro)
@@ -15,16 +15,15 @@
       <material name="drqp_black"/>
     </visual>
-    <!-- TODO: Define later -->
-    <!-- <collision>
-      <origin rpy="0 0 0" xyz="0 0 0"/>
-      <geometry>
-        <mesh filename="package://drqp_description/meshes/servo.stl" />
-      </geometry>
-    </collision>
-    <inertial>
-      <origin rpy="0 0 0" xyz="0.019066 -0.000002 0.006577"/>
-      <mass value="0.02471" />
-      <inertia ixx="0.0000215400" iyy="0.00002657000" izz="0.00002925000" ixy="-0.00000000122" ixz="-0.00000192741" iyz="-0.00000000001" />
-    </inertial> -->
+    <collision>
+      <origin xyz="0 0 0" rpy="0 0 ${-pi/2}" />
+      <geometry>
+        <mesh filename="package://drqp_description/meshes/servo.stl" />
+      </geometry>
+    </collision>
+    <inertial>
+      <origin rpy="0 0 0" xyz="0.019066 -0.000002 0.006577"/>
+      <mass value="0.02471" />
+      <inertia ixx="0.0000215400" iyy="0.00002657000" izz="0.00002925000" ixy="-0.00000000122" ixz="-0.00000192741" iyz="-0.00000000001" />
+    </inertial>
   </link>
   <joint name="${prefix}_coxa" type="revolute">
@@ -122,16 +121,15 @@
       <material name="drqp_black"/>
     </visual>
-    <!-- TODO: Define later -->
-    <!-- <collision>
-      <origin rpy="0 0 0" xyz="0 0 0"/>
-      <geometry>
-        <mesh filename="package://drqp_description/meshes/servo.stl" />
-      </geometry>
-    </collision>
-    <inertial>
-      <origin rpy="0 0 0" xyz="0.019066 -0.000002 0.006577"/>
-      <mass value="0.02471" />
-      <inertia ixx="0.0000215400" iyy="0.00002657000" izz="0.00002925000" ixy="-0.00000000122" ixz="-0.00000192741" iyz="-0.00000000001" />
-    </inertial> -->
+    <collision>
+      <origin rpy="0 ${pi/2} ${pi/2}" xyz="0 0 0" />
+      <geometry>
+        <mesh filename="package://drqp_description/meshes/servo.stl" />
+      </geometry>
+    </collision>
+    <inertial>
+      <origin rpy="0 0 0" xyz="0.019066 -0.000002 0.006577"/>
+      <mass value="0.02471" />
+      <inertia ixx="0.0000215400" iyy="0.00002657000" izz="0.00002925000" ixy="-0.00000000122" ixz="-0.00000192741" iyz="-0.00000000001" />
+    </inertial>
   </link>
   <joint name="${prefix}_femur_inner_1" type="fixed">
@@ -223,8 +221,6 @@
       <material name="drqp_black"/>
     </visual>
-    <!-- TODO: Define later -->
-    <!--
-    <collision>
-      <origin rpy="0 ${pi/2} ${pi/2}" xyz="0 0 0"" />
+    <collision>
+      <origin rpy="0 ${pi/2} ${pi/2}" xyz="0 0 0" />
       <geometry>
         <mesh filename="package://drqp_description/meshes/servo.stl" />
@@ -236,5 +232,4 @@
       <inertia ixx="0.0001762000" iyy="0.0005158000" izz="0.0003768000" ixy="-0.0000014522" ixz="0.0001789000" iyz="0.0000006181" />
     </inertial>
-    -->
   </link>
   <joint name="${prefix}_tibia_leg" type="fixed">

Commit message: stub all internal

File: src/drqp_description/urdf/leg.urdf.xacro (robot description, xacro)
@@ -1,4 +1,11 @@
 <?xml version="1.0"?>
 <robot xmlns:xacro="http://ros.org/wiki/xacro">
+  <xacro:include filename="$(find drqp_description)/urdf/inertial_macros.xacro"/>
+  <xacro:macro name="inertial_stub" params="">
+    <xacro:property name="tiny_value" value="0.0001"/>
+    <xacro:inertial_box mass="${tiny_value}" x="${tiny_value}" y="${tiny_value}" z="${tiny_value}">
+      <origin xyz="0 0 0" rpy="0 0 0"/>
+    </xacro:inertial_box>
+  </xacro:macro>
   <xacro:macro name="leg" params="robot_name prefix x y yaw">
   <joint name="${prefix}_coxa_servo" type="fixed">
@@ -57,11 +64,5 @@
       </geometry>
     </collision>
-    <!-- TODO: Define later -->
-    <!--
-    <inertial>
-      <origin rpy="0 0 0" xyz="0.019066 -0.000002 0.006577"/>
-      <mass value="0.02471" />
-      <inertia ixx="0.0000215400" iyy="0.00002657000" izz="0.00002925000" ixy="-0.00000000122" ixz="-0.00000192741" iyz="-0.00000000001" />
-    </inertial> -->
+    <xacro:inertial_stub />
   </link>
   <joint name="${prefix}_coxa_inner" type="fixed">
@@ -84,11 +85,5 @@
       </geometry>
     </collision>
-    <!-- TODO: Define later -->
-    <!--
-    <inertial>
-      <origin rpy="0 0 0" xyz="0.019066 -0.000002 0.006577"/>
-      <mass value="0.02471" />
-      <inertia ixx="0.0000215400" iyy="0.00002657000" izz="0.00002925000" ixy="-0.00000000122" ixz="-0.00000192741" iyz="-0.00000000001" />
-    </inertial> -->
+    <xacro:inertial_stub />
   </link>
   <joint name="${prefix}_femur" type="revolute">
@@ -156,11 +151,5 @@
       </geometry>
     </collision>
-    <!-- TODO: Define later -->
-    <!--
-    <inertial>
-      <origin rpy="0 0 0" xyz="0.020226 -0.00029 -0.00063"/>
-      <mass value="0.085834" />
-      <inertia ixx="0.0000288700" iyy="0.0000750200" izz="0.0000867200" ixy="0.0000002419" ixz="0.0000048494" iyz="0.0000000003" />
-    </inertial> -->
+    <xacro:inertial_stub />
   </link>
   <joint name="${prefix}_femur_inner_2" type="fixed">
@@ -188,11 +177,5 @@
       </geometry>
     </collision>
-    <!-- TODO: Define later -->
-    <!--
-    <inertial>
-      <origin rpy="0 0 0" xyz="0.020226 -0.00029 -0.00063"/>
-      <mass value="0.085834" />
-      <inertia ixx="0.0000288700" iyy="0.0000750200" izz="0.0000867200" ixy="0.0000002419" ixz="0.0000048494" iyz="0.0000000003" />
-    </inertial> -->
+    <xacro:inertial_stub />
   </link>
   <joint name="${prefix}_tibia" type="revolute">
@@ -255,11 +238,5 @@
       </geometry>
     </collision>
-    <!-- TODO: Define later -->
-    <!--
-    <inertial>
-      <origin rpy="0 0 0" xyz="0.020226 -0.00029 -0.00063"/>
-      <mass value="0.085834" />
-      <inertia ixx="0.0000288700" iyy="0.0000750200" izz="0.0000867200" ixy="0.0000002419" ixz="0.0000048494" iyz="0.0000000003" />
-    </inertial> -->
+    <xacro:inertial_stub />
   </link>
   <joint name="${prefix}_foot" type="fixed">

Commit message: model loads in gazebo

File: src/drqp_description/urdf/leg.urdf.xacro (robot description, xacro)
@@ -3,5 +3,5 @@
   <xacro:include filename="$(find drqp_description)/urdf/inertial_macros.xacro"/>
   <xacro:macro name="inertial_stub" params="">
-    <xacro:property name="tiny_value" value="0.0001"/>
+    <xacro:property name="tiny_value" value="0.01"/>
     <xacro:inertial_box mass="${tiny_value}" x="${tiny_value}" y="${tiny_value}" z="${tiny_value}">
       <origin xyz="0 0 0" rpy="0 0 0"/>
@@ -14,4 +14,7 @@
     <child link="${robot_name}/${prefix}_coxa_servo"/>
   </joint>
+  <gazebo reference='${prefix}_coxa_servo'>
+    <preserveFixedJoint>true</preserveFixedJoint>
+  </gazebo>
   <link name="${robot_name}/${prefix}_coxa_servo">
     <visual>
@@ -71,4 +74,7 @@
     <child link="${robot_name}/${prefix}_coxa_f2_link_2"/>
   </joint>
+  <gazebo reference='${prefix}_coxa_inner'>
+    <preserveFixedJoint>true</preserveFixedJoint>
+  </gazebo>
   <link name="${robot_name}/${prefix}_coxa_f2_link_2">
     <visual>
@@ -133,4 +139,7 @@
     <child link="${robot_name}/${prefix}_femur_link_f3"/>
   </joint>
+  <gazebo reference='${prefix}_femur_inner_1'>
+    <preserveFixedJoint>true</preserveFixedJoint>
+  </gazebo>
   <link name="${robot_name}/${prefix}_femur_link_f3">
     <visual>
@@ -158,4 +167,7 @@
     <child link="${robot_name}/${prefix}_femur_link_f1"/>
   </joint>
+  <gazebo reference='${prefix}_femur_inner_2'>
+    <preserveFixedJoint>true</preserveFixedJoint>
+  </gazebo>
   <link name="${robot_name}/${prefix}_femur_link_f1">
     <visual>
@@ -221,4 +233,7 @@
     <child link="${robot_name}/${prefix}_tibia_leg"/>
   </joint>
+  <gazebo reference='${prefix}_tibia_leg'>
+    <preserveFixedJoint>true</preserveFixedJoint>
+  </gazebo>
   <link name="${robot_name}/${prefix}_tibia_leg">
     <visual>
@@ -245,4 +260,7 @@
     <child link="${robot_name}/${prefix}_foot_link"/>
   </joint>
+  <gazebo reference='${prefix}_foot'>
+    <preserveFixedJoint>true</preserveFixedJoint>
+  </gazebo>
   <link name="${robot_name}/${prefix}_foot_link"/>
 </xacro:macro>

Commit message: turn off friction as it creates crazy dance in gazebo

File: src/drqp_description/urdf/leg.urdf.xacro (robot description, xacro)
@@ -42,5 +42,5 @@
     <parent link="${robot_name}/${prefix}_coxa_servo"/>
     <child link="${robot_name}/${prefix}_coxa_f2_link_1"/>
-    <dynamics friction="0.5"/>
+    <!-- <dynamics friction="5"/> -->
   </joint>
   <transmission name="trans_${prefix}_coxa">
@@ -99,5 +99,5 @@
     <parent link="${robot_name}/${prefix}_coxa_f2_link_2"/>
     <child link="${robot_name}/${prefix}_femur_servo"/>
-    <dynamics friction="0.5"/>
+    <!-- <dynamics friction="5"/> -->
   </joint>
   <transmission name="trans_${prefix}_femur">
@@ -197,5 +197,5 @@
     <parent link="${robot_name}/${prefix}_femur_link_f1"/>
     <child link="${robot_name}/${prefix}_tibia_servo"/>
-    <dynamics friction="0.5"/>
+    <!-- <dynamics friction="5"/> -->
   </joint>
   <transmission name="trans_${prefix}_tibia">

Commit message: non hanging damping

File: src/drqp_description/urdf/leg.urdf.xacro (robot description, xacro)
@@ -42,6 +42,9 @@
     <parent link="${robot_name}/${prefix}_coxa_servo"/>
     <child link="${robot_name}/${prefix}_coxa_f2_link_1"/>
-    <!-- <dynamics friction="5"/> -->
-  </joint>
+    <!-- <dynamics damping="100" friction="0.1" /> -->
+  </joint>
+  <gazebo reference="${prefix}_coxa">
+    <dampingFactor>0.2</dampingFactor>
+  </gazebo>
   <transmission name="trans_${prefix}_coxa">
     <type>transmission_interface/SimpleTransmission</type>
@@ -99,6 +102,9 @@
     <parent link="${robot_name}/${prefix}_coxa_f2_link_2"/>
     <child link="${robot_name}/${prefix}_femur_servo"/>
-    <!-- <dynamics friction="5"/> -->
-  </joint>
+    <!-- <dynamics damping="100" friction="0.1" /> -->
+  </joint>
+  <gazebo reference="${prefix}_femur">
+    <dampingFactor>0.2</dampingFactor>
+  </gazebo>
   <transmission name="trans_${prefix}_femur">
     <type>transmission_interface/SimpleTransmission</type>
@@ -197,6 +203,9 @@
     <parent link="${robot_name}/${prefix}_femur_link_f1"/>
     <child link="${robot_name}/${prefix}_tibia_servo"/>
-    <!-- <dynamics friction="5"/> -->
-  </joint>
+    <!-- <dynamics damping="100" friction="0.1" /> -->
+  </joint>
+  <gazebo reference="${prefix}_tibia">
+    <dampingFactor>0.2</dampingFactor>
+  </gazebo>
   <transmission name="trans_${prefix}_tibia">
     <type>transmission_interface/SimpleTransmission</type>

Commit message: joints need prefixes

File: src/drqp_description/urdf/leg.urdf.xacro (robot description, xacro)
@@ -9,5 +9,5 @@
   </xacro:macro>
   <xacro:macro name="leg" params="robot_name prefix x y yaw">
-  <joint name="${prefix}_coxa_servo" type="fixed">
+  <joint name="${robot_name}/${prefix}_coxa_servo" type="fixed">
     <origin rpy="0 0 ${yaw}" xyz="${x} ${y} 0"/>
     <parent link="${robot_name}/base_center_link"/>
@@ -37,5 +37,5 @@
     </inertial>
   </link>
-  <joint name="${prefix}_coxa" type="revolute">
+  <joint name="${robot_name}/${prefix}_coxa" type="revolute">
     <axis xyz="0 0 1"/>
     <limit effort="3" lower="${radians(-90)}" upper="${radians(90)}" velocity="${pi}"/>
@@ -66,5 +66,5 @@
     <xacro:inertial_stub />
   </link>
-  <joint name="${prefix}_coxa_inner" type="fixed">
+  <joint name="${robot_name}/${prefix}_coxa_inner" type="fixed">
     <origin rpy="0 0 0" xyz="${0.0265 * 2} 0 0"/>
     <parent link="${robot_name}/${prefix}_coxa_f2_link_1"/>
@@ -90,5 +90,5 @@
     <xacro:inertial_stub />
   </link>
-  <joint name="${prefix}_femur" type="revolute">
+  <joint name="${robot_name}/${prefix}_femur" type="revolute">
     <axis xyz="0 1 0"/>
     <limit effort="3" lower="${radians(-98)}" upper="${radians(90)}" velocity="${pi}"/>
@@ -128,5 +128,5 @@
     </inertial>
   </link>
-  <joint name="${prefix}_femur_inner_1" type="fixed">
+  <joint name="${robot_name}/${prefix}_femur_inner_1" type="fixed">
     <origin rpy="0 0 0" xyz="${0.036 + 0.0055} 0 0"/>
     <parent link="${robot_name}/${prefix}_femur_servo"/>
@@ -156,5 +156,5 @@
     <xacro:inertial_stub />
   </link>
-  <joint name="${prefix}_femur_inner_2" type="fixed">
+  <joint name="${robot_name}/${prefix}_femur_inner_2" type="fixed">
     <origin rpy="0 0 0" xyz="0.023 0 -0.015"/>
     <parent link="${robot_name}/${prefix}_femur_link_f3"/>
@@ -185,5 +185,5 @@
     <xacro:inertial_stub />
   </link>
-  <joint name="${prefix}_tibia" type="revolute">
+  <joint name="${robot_name}/${prefix}_tibia" type="revolute">
     <axis xyz="0 1 0"/>
     <limit effort="3" lower="${radians(-125)}" upper="${radians(80)}" velocity="${pi}"/>
@@ -219,5 +219,5 @@
     </inertial>
   </link>
-  <joint name="${prefix}_tibia_leg" type="fixed">
+  <joint name="${robot_name}/${prefix}_tibia_leg" type="fixed">
     <origin rpy="0 0 0" xyz="0.0325 0 0"/>
     <parent link="${robot_name}/${prefix}_tibia_servo"/>
@@ -246,5 +246,5 @@
     <xacro:inertial_stub />
   </link>
-  <joint name="${prefix}_foot" type="fixed">
+  <joint name="${robot_name}/${prefix}_foot" type="fixed">
     <origin rpy="0 0 0" xyz="0.052797 0 -0.088395"/>
     <parent link="${robot_name}/${prefix}_tibia_leg"/>
