Commit message: put robot above the ground

File: packages/runtime/drqp_description/urdf/body.urdf.xacro (robot description, xacro)
@@ -22,6 +22,5 @@
     </inertial>
   </link>
-  <link name="$(arg robot_name)/base_link"> <!-- AKA World -->
-  </link>
+  <link name="$(arg robot_name)/base_link" /> <!-- Robot base lowest point -->
   <joint name="base_bottom" type="fixed">
     <origin rpy="0 0 0" xyz="0 0 ${body_height/2}"/>

File: packages/runtime/drqp_description/urdf/dr_qp.urdf.xacro (robot description, xacro)
@@ -12,4 +12,5 @@
     <color rgba="0.5 0.5 0.5 0.2" />
   </material>
+  <xacro:property name="robot_height" value="0.085" />
   <xacro:include filename="$(find drqp_description)/urdf/body.urdf.xacro"/>
   <xacro:include filename="$(find drqp_description)/urdf/leg.urdf.xacro"/>
@@ -21,4 +22,10 @@
   <xacro:leg robot_name="$(arg robot_name)" prefix="left_middle" x="0" y="0.103" yaw="${pi/2}"/>
   <xacro:leg robot_name="$(arg robot_name)" prefix="left_back" x="-0.11692" y="0.06387" yaw="${3*pi/4}"/>
+  <link name="world" />
+  <joint name="world_to_base_link=" type="fixed">
+      <origin rpy="0 0 0" xyz="0 0 ${robot_height}"/>
+      <parent link="world"/>
+      <child link="$(arg robot_name)/base_link"/>
+  </joint>
   <gazebo reference="">
     <self_collide>1</self_collide>
