Commit message: adjust leg angles

File: packages/runtime/drqp_description/urdf/leg.urdf.xacro (robot description, xacro)
@@ -187,5 +187,5 @@
   <joint name="${robot_name}/${prefix}_tibia" type="revolute">
     <axis xyz="0 1 0"/>
-    <limit effort="3" lower="${radians(-125)}" upper="${radians(80)}" velocity="${pi}"/>
+    <limit effort="3" lower="${radians(-80)}" upper="${radians(110)}" velocity="${pi}"/>
     <origin rpy="0 0 0" xyz="0 0 0"/>
     <parent link="${robot_name}/${prefix}_femur_link_f1"/>

Commit message: fix duplicate names

File: packages/runtime/drqp_description/urdf/leg.urdf.xacro (robot description, xacro)
@@ -9,5 +9,5 @@
   </xacro:macro>
   <xacro:macro name="leg" params="robot_name prefix x y yaw">
-  <joint name="${robot_name}/${prefix}_coxa_servo" type="fixed">
+  <joint name="${robot_name}/${prefix}_coxa_servo_joint" type="fixed">
     <origin rpy="0 0 ${yaw}" xyz="${x} ${y} 0"/>
     <parent link="${robot_name}/base_center_link"/>
@@ -207,5 +207,5 @@
     </inertial>
   </link>
-  <joint name="${robot_name}/${prefix}_tibia_leg" type="fixed">
+  <joint name="${robot_name}/${prefix}_tibia_leg_joint" type="fixed">
     <origin rpy="0 0 0" xyz="0.0325 0 0"/>
     <parent link="${robot_name}/${prefix}_tibia_servo"/>
