Commit message: break out node from robot config make robot config usable without reading yml config

File: packages/runtime/drqp_description/urdf/ros2_control.urdf.xacro (robot description, xacro)
@@ -1,7 +1,8 @@
 <?xml version="1.0"?>
 <robot xmlns:xacro="http://www.ros.org/wiki/xacro">
-  <xacro:macro name="drqp_leg_ros2_control" params="robot_name leg_name">
+  <xacro:macro name="drqp_leg_ros2_control" params="robot_name leg_name coxa_servo_id servo_inverted">
     <joint name="${robot_name}/${leg_name}_coxa">
       <command_interface name="position">
+        <param name="servo_id">${coxa_servo_id}</param>
         <param name="min">${radians(-90)}</param>
         <param name="max">${radians(90)}</param>
@@ -11,4 +12,6 @@
     <joint name="${robot_name}/${leg_name}_femur">
       <command_interface name="position">
+        <param name="servo_id">${coxa_servo_id + 2}</param>
+        <param name="inverted">${servo_inverted}</param>
         <param name="min">${radians(-98)}</param>
         <param name="max">${radians(90)}</param>
@@ -18,4 +21,6 @@
     <joint name="${robot_name}/${leg_name}_tibia">
       <command_interface name="position">
+        <param name="servo_id">${coxa_servo_id + 4}</param>
+        <param name="inverted">${servo_inverted}</param>
         <param name="min">${radians(-80)}</param>
         <param name="max">${radians(110)}</param>
@@ -28,11 +33,13 @@
       <hardware>
         <plugin>drqp_control/a1_16_hardware_interface</plugin>
+        <param name="device_address">/dev/ttySC0</param>
+        <param name="baud_rate">115200</param>
       </hardware>
-      <xacro:drqp_leg_ros2_control robot_name="${robot_name}" leg_name="left_front"/>
-      <xacro:drqp_leg_ros2_control robot_name="${robot_name}" leg_name="right_front"/>
-      <xacro:drqp_leg_ros2_control robot_name="${robot_name}" leg_name="left_middle"/>
-      <xacro:drqp_leg_ros2_control robot_name="${robot_name}" leg_name="right_middle"/>
-      <xacro:drqp_leg_ros2_control robot_name="${robot_name}" leg_name="left_back"/>
-      <xacro:drqp_leg_ros2_control robot_name="${robot_name}" leg_name="right_back"/>
+      <xacro:drqp_leg_ros2_control robot_name="${robot_name}" leg_name="left_front" coxa_servo_id="1"/>
+      <xacro:drqp_leg_ros2_control robot_name="${robot_name}" leg_name="right_front" coxa_servo_id="2" servo_inverted="true"/>
+      <xacro:drqp_leg_ros2_control robot_name="${robot_name}" leg_name="left_middle" coxa_servo_id="13"/>
+      <xacro:drqp_leg_ros2_control robot_name="${robot_name}" leg_name="right_middle" coxa_servo_id="14" servo_inverted="true"/>
+      <xacro:drqp_leg_ros2_control robot_name="${robot_name}" leg_name="left_back" coxa_servo_id="7"/>
+      <xacro:drqp_leg_ros2_control robot_name="${robot_name}" leg_name="right_back" coxa_servo_id="8" servo_inverted="true"/>
     </ros2_control>
   </xacro:macro>

Commit message: fix xml

File: packages/runtime/drqp_description/urdf/ros2_control.urdf.xacro (robot description, xacro)
@@ -1,5 +1,5 @@
 <?xml version="1.0"?>
 <robot xmlns:xacro="http://www.ros.org/wiki/xacro">
-  <xacro:macro name="drqp_leg_ros2_control" params="robot_name leg_name coxa_servo_id servo_inverted">
+  <xacro:macro name="drqp_leg_ros2_control" params="robot_name leg_name coxa_servo_id servo_inverted:=false">
     <joint name="${robot_name}/${leg_name}_coxa">
       <command_interface name="position">

Commit message: implement pose setting in the hardware interface

File: packages/runtime/drqp_description/urdf/ros2_control.urdf.xacro (robot description, xacro)
@@ -1,10 +1,12 @@
 <?xml version="1.0"?>
 <robot xmlns:xacro="http://www.ros.org/wiki/xacro">
-  <xacro:macro name="drqp_leg_ros2_control" params="robot_name leg_name coxa_servo_id servo_inverted:=false">
+  <xacro:macro name="drqp_leg_ros2_control" params="robot_name leg_name coxa_servo_id servo_inverted:=false offset_coxa:=0.0 offset_femur:=0.0 offset_tibia:=0.0">
     <joint name="${robot_name}/${leg_name}_coxa">
       <command_interface name="position">
         <param name="servo_id">${coxa_servo_id}</param>
+        <param name="inverted">false</param>
         <param name="min">${radians(-90)}</param>
         <param name="max">${radians(90)}</param>
+        <param name="offset_rads">${offset_coxa}</param>
       </command_interface>
       <state_interface name="position"/>
@@ -16,4 +18,5 @@
         <param name="min">${radians(-98)}</param>
         <param name="max">${radians(90)}</param>
+        <param name="offset_rads">${offset_femur}</param>
       </command_interface>
       <state_interface name="position"/>
@@ -25,4 +28,5 @@
         <param name="min">${radians(-80)}</param>
         <param name="max">${radians(110)}</param>
+        <param name="offset_rads">${offset_tibia}</param>
       </command_interface>
       <state_interface name="position"/>

Commit message: fix bool param

File: packages/runtime/drqp_description/urdf/ros2_control.urdf.xacro (robot description, xacro)
@@ -1,9 +1,9 @@
 <?xml version="1.0"?>
 <robot xmlns:xacro="http://www.ros.org/wiki/xacro">
-  <xacro:macro name="drqp_leg_ros2_control" params="robot_name leg_name coxa_servo_id servo_inverted:=false offset_coxa:=0.0 offset_femur:=0.0 offset_tibia:=0.0">
+  <xacro:macro name="drqp_leg_ros2_control" params="robot_name leg_name coxa_servo_id servo_inverted:=False offset_coxa:=0.0 offset_femur:=0.0 offset_tibia:=0.0">
     <joint name="${robot_name}/${leg_name}_coxa">
       <command_interface name="position">
         <param name="servo_id">${coxa_servo_id}</param>
-        <param name="inverted">false</param>
+        <param name="inverted">False</param>
         <param name="min">${radians(-90)}</param>
         <param name="max">${radians(90)}</param>
@@ -41,9 +41,9 @@
       </hardware>
       <xacro:drqp_leg_ros2_control robot_name="${robot_name}" leg_name="left_front" coxa_servo_id="1"/>
-      <xacro:drqp_leg_ros2_control robot_name="${robot_name}" leg_name="right_front" coxa_servo_id="2" servo_inverted="true"/>
+      <xacro:drqp_leg_ros2_control robot_name="${robot_name}" leg_name="right_front" coxa_servo_id="2" servo_inverted="True"/>
       <xacro:drqp_leg_ros2_control robot_name="${robot_name}" leg_name="left_middle" coxa_servo_id="13"/>
-      <xacro:drqp_leg_ros2_control robot_name="${robot_name}" leg_name="right_middle" coxa_servo_id="14" servo_inverted="true"/>
+      <xacro:drqp_leg_ros2_control robot_name="${robot_name}" leg_name="right_middle" coxa_servo_id="14" servo_inverted="True"/>
       <xacro:drqp_leg_ros2_control robot_name="${robot_name}" leg_name="left_back" coxa_servo_id="7"/>
-      <xacro:drqp_leg_ros2_control robot_name="${robot_name}" leg_name="right_back" coxa_servo_id="8" servo_inverted="true"/>
+      <xacro:drqp_leg_ros2_control robot_name="${robot_name}" leg_name="right_back" coxa_servo_id="8" servo_inverted="True"/>
     </ros2_control>
   </xacro:macro>

Commit message: set max torque to 20%

File: packages/runtime/drqp_description/urdf/ros2_control.urdf.xacro (robot description, xacro)
@@ -1,12 +1,13 @@
 <?xml version="1.0"?>
 <robot xmlns:xacro="http://www.ros.org/wiki/xacro">
-  <xacro:macro name="drqp_leg_ros2_control" params="robot_name leg_name coxa_servo_id servo_inverted:=False offset_coxa:=0.0 offset_femur:=0.0 offset_tibia:=0.0">
+  <xacro:macro name="drqp_leg_ros2_control" params="robot_name leg_name coxa_servo_id servo_inverted:=False offset_coxa:=0.0 offset_femur:=0.0 offset_tibia:=0.0 max_torque:=0.2">
     <joint name="${robot_name}/${leg_name}_coxa">
       <command_interface name="position">
         <param name="servo_id">${coxa_servo_id}</param>
         <param name="inverted">False</param>
+        <param name="offset_rads">${offset_coxa}</param>
+        <param name="max_torque">${max_torque}</param>
         <param name="min">${radians(-90)}</param>
         <param name="max">${radians(90)}</param>
-        <param name="offset_rads">${offset_coxa}</param>
         <param name="initial_value">0.0</param> <!-- Initial value for mock_hardware -->
       </command_interface>
@@ -20,7 +21,8 @@
         <param name="servo_id">${coxa_servo_id + 2}</param>
         <param name="inverted">${servo_inverted}</param>
+        <param name="offset_rads">${offset_femur}</param>
+        <param name="max_torque">${max_torque}</param>
         <param name="min">${radians(-98)}</param>
         <param name="max">${radians(90)}</param>
-        <param name="offset_rads">${offset_femur}</param>
         <param name="initial_value">0.0</param> <!-- Initial value for mock_hardware -->
       </command_interface>
@@ -34,7 +36,8 @@
         <param name="servo_id">${coxa_servo_id + 4}</param>
         <param name="inverted">${servo_inverted}</param>
+        <param name="offset_rads">${offset_coxa}</param>
+        <param name="max_torque">${max_torque}</param>
         <param name="min">${radians(-80)}</param>
         <param name="max">${radians(110)}</param>
-        <param name="offset_rads">${offset_tibia}</param>
         <param name="initial_value">0.0</param> <!-- Initial value for mock_hardware -->
       </command_interface>

Commit message: 0.5 torque log configure

File: packages/runtime/drqp_description/urdf/ros2_control.urdf.xacro (robot description, xacro)
@@ -1,5 +1,5 @@
 <?xml version="1.0"?>
 <robot xmlns:xacro="http://www.ros.org/wiki/xacro">
-  <xacro:macro name="drqp_leg_ros2_control" params="robot_name leg_name coxa_servo_id servo_inverted:=False offset_coxa:=0.0 offset_femur:=0.0 offset_tibia:=0.0 max_torque:=0.2">
+  <xacro:macro name="drqp_leg_ros2_control" params="robot_name leg_name coxa_servo_id servo_inverted:=False offset_coxa:=0.0 offset_femur:=0.0 offset_tibia:=0.0 max_torque:=0.5">
     <joint name="${robot_name}/${leg_name}_coxa">
       <command_interface name="position">

Commit message: 25% torque

File: packages/runtime/drqp_description/urdf/ros2_control.urdf.xacro (robot description, xacro)
@@ -1,5 +1,5 @@
 <?xml version="1.0"?>
 <robot xmlns:xacro="http://www.ros.org/wiki/xacro">
-  <xacro:macro name="drqp_leg_ros2_control" params="robot_name leg_name coxa_servo_id servo_inverted:=False offset_coxa:=0.0 offset_femur:=0.0 offset_tibia:=0.0 max_torque:=0.5">
+  <xacro:macro name="drqp_leg_ros2_control" params="robot_name leg_name coxa_servo_id servo_inverted:=False offset_coxa:=0.0 offset_femur:=0.0 offset_tibia:=0.0 max_torque:=0.25">
     <joint name="${robot_name}/${leg_name}_coxa">
       <command_interface name="position">
