Commit message: Configure servo limits on startup (#243)
Add torque setting to URDF and RobotConfig. Default to 25% in URDF and
100% in C++
Apply max torque, min position and max position for all servos at
startup

Other changes:
Add setter for min/max position in XYZServo
Use `offsetof()` for all offsets in ram/eeprom setters/getters in
XYZServo. No more magic numbers.

---------

Co-authored-by: anton-matosov <3339485+anton-matosov@users.noreply.github.com>
Co-authored-by: Copilot Autofix powered by AI <62310815+github-advanced-security[bot]@users.noreply.github.com>

File: packages/runtime/drqp_description/urdf/ros2_control.urdf.xacro (robot description, xacro)
@@ -1,12 +1,13 @@
 <?xml version="1.0"?>
 <robot xmlns:xacro="http://www.ros.org/wiki/xacro">
-  <xacro:macro name="drqp_leg_ros2_control" params="robot_name leg_name coxa_servo_id servo_inverted:=False offset_coxa:=0.0 offset_femur:=0.0 offset_tibia:=0.0">
+  <xacro:macro name="drqp_leg_ros2_control" params="robot_name leg_name coxa_servo_id servo_inverted:=False offset_coxa:=0.0 offset_femur:=0.0 offset_tibia:=0.0 max_torque:=0.25">
     <joint name="${robot_name}/${leg_name}_coxa">
       <command_interface name="position">
         <param name="servo_id">${coxa_servo_id}</param>
         <param name="inverted">False</param>
+        <param name="offset_rads">${offset_coxa}</param>
+        <param name="max_torque">${max_torque}</param>
         <param name="min">${radians(-90)}</param>
         <param name="max">${radians(90)}</param>
-        <param name="offset_rads">${offset_coxa}</param>
         <param name="initial_value">0.0</param> <!-- Initial value for mock_hardware -->
       </command_interface>
@@ -20,7 +21,8 @@
         <param name="servo_id">${coxa_servo_id + 2}</param>
         <param name="inverted">${servo_inverted}</param>
+        <param name="offset_rads">${offset_femur}</param>
+        <param name="max_torque">${max_torque}</param>
         <param name="min">${radians(-98)}</param>
         <param name="max">${radians(90)}</param>
-        <param name="offset_rads">${offset_femur}</param>
         <param name="initial_value">0.0</param> <!-- Initial value for mock_hardware -->
       </command_interface>
@@ -34,7 +36,8 @@
         <param name="servo_id">${coxa_servo_id + 4}</param>
         <param name="inverted">${servo_inverted}</param>
+        <param name="offset_rads">${offset_tibia}</param>
+        <param name="max_torque">${max_torque}</param>
         <param name="min">${radians(-80)}</param>
         <param name="max">${radians(110)}</param>
-        <param name="offset_rads">${offset_tibia}</param>
         <param name="initial_value">0.0</param> <!-- Initial value for mock_hardware -->
       </command_interface>
