Commit message: split jsp from rviz

File: packages/runtime/drqp_description/urdf/dr_qp.urdf.xacro (robot description, xacro)
@@ -2,7 +2,5 @@
 <robot name="dr_qp" xmlns:xacro="http://ros.org/wiki/xacro">
   <xacro:arg name="robot_name" default = "dr_qp"/>
-  <xacro:arg name="external_urdf_loc" default=""/>
   <xacro:arg name="load_gazebo_configs" default="false"/>
-  <xacro:property name="urdf_loc" value="$(arg external_urdf_loc)"/>
   <xacro:if value="$(arg load_gazebo_configs)">
     <xacro:include filename="$(find drqp_gazebo)/config/drqp_texture.gazebo"/>

Commit message: Fixup robot description in URDF (#118)
Fix launch files to make them easier to use and more readable
Add world link and raise robot above it to the appropriate height so
that feet start on the ground
Update rviz config to match new reality

Update hexapod_js launch files to have more readable code there

File: packages/runtime/drqp_description/urdf/dr_qp.urdf.xacro (robot description, xacro)
@@ -2,7 +2,5 @@
 <robot name="dr_qp" xmlns:xacro="http://ros.org/wiki/xacro">
   <xacro:arg name="robot_name" default = "dr_qp"/>
-  <xacro:arg name="external_urdf_loc" default=""/>
   <xacro:arg name="load_gazebo_configs" default="false"/>
-  <xacro:property name="urdf_loc" value="$(arg external_urdf_loc)"/>
   <xacro:if value="$(arg load_gazebo_configs)">
     <xacro:include filename="$(find drqp_gazebo)/config/drqp_texture.gazebo"/>
@@ -14,4 +12,5 @@
     <color rgba="0.5 0.5 0.5 0.2" />
   </material>
+  <xacro:property name="robot_height" value="0.085" />
   <xacro:include filename="$(find drqp_description)/urdf/body.urdf.xacro"/>
   <xacro:include filename="$(find drqp_description)/urdf/leg.urdf.xacro"/>
@@ -23,4 +22,10 @@
   <xacro:leg robot_name="$(arg robot_name)" prefix="left_middle" x="0" y="0.103" yaw="${pi/2}"/>
   <xacro:leg robot_name="$(arg robot_name)" prefix="left_back" x="-0.11692" y="0.06387" yaw="${3*pi/4}"/>
+  <link name="world" />
+  <joint name="world_to_base_link=" type="fixed">
+      <origin rpy="0 0 0" xyz="0 0 ${robot_height}"/>
+      <parent link="world"/>
+      <child link="$(arg robot_name)/base_link"/>
+  </joint>
   <gazebo reference="">
     <self_collide>1</self_collide>

Commit message: setup ros2_control interfaces the right way

File: packages/runtime/drqp_description/urdf/dr_qp.urdf.xacro (robot description, xacro)
@@ -28,4 +28,6 @@
       <child link="$(arg robot_name)/base_link"/>
   </joint>
+  <xacro:include filename="$(find drqp_description)/urdf/ros2_control.urdf.xacro"/>
+  <xacro:drqp_ros2_control robot_name="$(arg robot_name)" />
   <gazebo reference="">
     <self_collide>1</self_collide>

File: packages/runtime/drqp_description/urdf/leg.urdf.xacro (robot description, xacro)
@@ -255,6 +255,4 @@
   </gazebo>
   <link name="${robot_name}/${prefix}_foot_link"/>
-  <xacro:include filename="$(find drqp_description)/urdf/ros2_control.urdf.xacro"/>
-  <xacro:drqp_ros2_control robot_name="${robot_name}" prefix="${prefix}"/>
 </xacro:macro>
 </robot>

File: packages/runtime/drqp_description/urdf/ros2_control.urdf.xacro (robot description, xacro)
@@ -1,30 +1,38 @@
 <?xml version="1.0"?>
 <robot xmlns:xacro="http://www.ros.org/wiki/xacro">
-  <xacro:macro name="drqp_ros2_control" params="robot_name prefix">
-    <ros2_control name="${robot_name}_${prefix}" type="system">
+  <xacro:macro name="drqp_leg_ros2_control" params="robot_name leg_name">
+    <joint name="${robot_name}/${leg_name}_coxa">
+      <command_interface name="position">
+        <param name="min">${radians(-90)}</param>
+        <param name="max">${radians(90)}</param>
+      </command_interface>
+      <state_interface name="position"/>
+    </joint>
+    <joint name="${robot_name}/${leg_name}_femur">
+      <command_interface name="position">
+        <param name="min">${radians(-98)}</param>
+        <param name="max">${radians(90)}</param>
+      </command_interface>
+      <state_interface name="position"/>
+    </joint>
+    <joint name="${robot_name}/${leg_name}_tibia">
+      <command_interface name="position">
+        <param name="min">${radians(-80)}</param>
+        <param name="max">${radians(110)}</param>
+      </command_interface>
+      <state_interface name="position"/>
+    </joint>
+  </xacro:macro>
+  <xacro:macro name="drqp_ros2_control" params="robot_name">
+    <ros2_control name="${robot_name}" type="system">
       <hardware>
         <plugin>drqp_control/a1_16_hardware_interface</plugin>
       </hardware>
-      <joint name="${robot_name}/${prefix}_coxa">
-        <command_interface name="position">
-          <param name="min">${radians(-90)}</param>
-          <param name="max">${radians(90)}</param>
-        </command_interface>
-        <state_interface name="position"/>
-      </joint>
-      <joint name="${robot_name}/${prefix}_femur">
-        <command_interface name="position">
-          <param name="min">${radians(-98)}</param>
-          <param name="max">${radians(90)}</param>
-        </command_interface>
-        <state_interface name="position"/>
-      </joint>
-      <joint name="${robot_name}/${prefix}_tibia">
-        <command_interface name="position">
-          <param name="min">${radians(-80)}</param>
-          <param name="max">${radians(110)}</param>
-        </command_interface>
-        <state_interface name="position"/>
-      </joint>
+      <xacro:drqp_leg_ros2_control robot_name="${robot_name}" leg_name="left_front"/>
+      <xacro:drqp_leg_ros2_control robot_name="${robot_name}" leg_name="right_front"/>
+      <xacro:drqp_leg_ros2_control robot_name="${robot_name}" leg_name="left_middle"/>
+      <xacro:drqp_leg_ros2_control robot_name="${robot_name}" leg_name="right_middle"/>
+      <xacro:drqp_leg_ros2_control robot_name="${robot_name}" leg_name="left_back"/>
+      <xacro:drqp_leg_ros2_control robot_name="${robot_name}" leg_name="right_back"/>
     </ros2_control>
   </xacro:macro>

Commit message: wire in device name through xacro, use it in test

File: packages/runtime/drqp_description/urdf/dr_qp.urdf.xacro (robot description, xacro)
@@ -3,4 +3,5 @@
   <xacro:arg name="robot_name" default = "dr_qp"/>
   <xacro:arg name="load_gazebo_configs" default="false"/>
+  <xacro:arg name="hardware_device_address" default="/dev/ttySC0"/>
   <xacro:if value="$(arg load_gazebo_configs)">
     <xacro:include filename="$(find drqp_gazebo)/config/drqp_texture.gazebo"/>
@@ -29,5 +30,5 @@
   </joint>
   <xacro:include filename="$(find drqp_description)/urdf/ros2_control.urdf.xacro"/>
-  <xacro:drqp_ros2_control robot_name="$(arg robot_name)" />
+  <xacro:drqp_ros2_control robot_name="$(arg robot_name)" device_address="$(arg hardware_device_address)" />
   <gazebo reference="">
     <self_collide>1</self_collide>

File: packages/runtime/drqp_description/urdf/ros2_control.urdf.xacro (robot description, xacro)
@@ -42,9 +42,9 @@
     </joint>
   </xacro:macro>
-  <xacro:macro name="drqp_ros2_control" params="robot_name">
+  <xacro:macro name="drqp_ros2_control" params="robot_name device_address:=/dev/ttySC0">
     <ros2_control name="${robot_name}" type="system" rw_rate="20" is_async="true" thread_priority="30">
       <hardware>
         <plugin>drqp_control/a1_16_hardware_interface</plugin>
-        <param name="device_address">/dev/ttySC0</param>
+        <param name="device_address">${device_address}</param>
         <param name="baud_rate">115200</param>
       </hardware>

Commit message: Pass in use_gazebo param Setup hardware for new sim Cleanup old gazebo placeholders

File: packages/runtime/drqp_description/urdf/dr_qp.urdf.xacro (robot description, xacro)
@@ -2,9 +2,6 @@
 <robot name="dr_qp" xmlns:xacro="http://ros.org/wiki/xacro">
   <xacro:arg name="robot_name" default = "dr_qp"/>
-  <xacro:arg name="load_gazebo_configs" default="false"/>
   <xacro:arg name="hardware_device_address" default="/dev/ttySC0"/>
-  <xacro:if value="$(arg load_gazebo_configs)">
-    <xacro:include filename="$(find drqp_gazebo)/config/drqp_texture.gazebo"/>
-  </xacro:if>
+  <xacro:arg name="use_gazebo" default="false" />
   <material name="drqp_black">
     <texture filename="package://drqp_description/meshes/drqp_black.png"/>
@@ -30,5 +27,5 @@
   </joint>
   <xacro:include filename="$(find drqp_description)/urdf/ros2_control.urdf.xacro"/>
-  <xacro:drqp_ros2_control robot_name="$(arg robot_name)" device_address="$(arg hardware_device_address)" />
+  <xacro:drqp_ros2_control robot_name="$(arg robot_name)" device_address="$(arg hardware_device_address)" use_gazebo="$(arg use_gazebo)" />
   <gazebo reference="">
     <self_collide>1</self_collide>

File: packages/runtime/drqp_description/urdf/gazebo.xacro (robot description, xacro)
@@ -1,46 +1,11 @@
 <?xml version="1.0"?>
 <robot xmlns:xacro="http://www.ros.org/wiki/xacro">
-    <ros2_control name="GazeboSystem" type="system">
-        <!-- <hardware> Fix in https://github.com/Dr-QP/Dr.QP/issues/91
-            <plugin>gazebo_ros2_control/GazeboSystem</plugin>
-        </hardware> -->
-        <xacro:macro name="hexjoint" params="name">
-            <joint name="${name}">
-                <command_interface name="position">
-                    <param name="min">-15</param>
-                    <param name="max">15</param>
-                </command_interface>
-                <state_interface name="position">
-                    <param name="initial_value">1.0</param>
-                </state_interface>
-                <state_interface name="velocity" />
-                <state_interface name="effort" />
-            </joint>
-        </xacro:macro>
-        <xacro:hexjoint name="left_back_coxa" />
-        <xacro:hexjoint name="left_back_femur" />
-        <xacro:hexjoint name="left_back_tibia" />
-        <!-- <xacro:hexjoint name="left_middle_coxa" /> -->
-        <!-- <xacro:hexjoint name="left_middle_femur" /> -->
-        <!-- <xacro:hexjoint name="left_middle_tibia" /> -->
-        <!-- <xacro:hexjoint name="left_front_coxa" /> -->
-        <!-- <xacro:hexjoint name="left_front_femur" /> -->
-        <!-- <xacro:hexjoint name="left_front_tibia" /> -->
-        <!-- <xacro:hexjoint name="right_front_coxa" /> -->
-        <!-- <xacro:hexjoint name="right_front_femur" /> -->
-        <!-- <xacro:hexjoint name="right_front_tibia" /> -->
-        <!-- <xacro:hexjoint name="right_middle_coxa" /> -->
-        <!-- <xacro:hexjoint name="right_middle_femur" /> -->
-        <!-- <xacro:hexjoint name="right_middle_tibia" /> -->
-        <!-- <xacro:hexjoint name="right_back_coxa" /> -->
-        <!-- <xacro:hexjoint name="right_back_femur" /> -->
-        <!-- <xacro:hexjoint name="right_back_tibia" /> -->
-    </ros2_control>
-    <!-- <gazebo> Fix in https://github.com/Dr-QP/Dr.QP/issues/91
-        <plugin filename="libgazebo_ros2_control.so" name="gazebo_ros2_control">
-          <robot_param>robot_description</robot_param>
-          <robot_param_node>robot_state_publisher</robot_param_node>
-          <parameters>$(find drqp_gazebo)/config/gazebo_params.yaml</parameters>
-        </plugin>
-    </gazebo> -->
+  <xacro:macro name="gazebo" params="robot_name">
+    <!-- Gazebo Classic definitions + plugin -->
+  <!-- <gazebo>
+    <plugin filename="gz_ros2_control-system" name="gz_ros2_control::GazeboSimROS2ControlPlugin">
+      <parameters>$(find drqp_control)/config/drqp_controllers.yaml</parameters>
+    </plugin>
+  </gazebo> -->
+  </xacro:macro>
 </robot>

File: packages/runtime/drqp_description/urdf/ros2_control.urdf.xacro (robot description, xacro)
@@ -45,10 +45,15 @@
     </joint>
   </xacro:macro>
-  <xacro:macro name="drqp_ros2_control" params="robot_name device_address:=/dev/ttySC0">
+  <xacro:macro name="drqp_ros2_control" params="robot_name device_address:=/dev/ttySC0 use_gazebo:=^|false">
     <ros2_control name="${robot_name}_servos" type="system" rw_rate="20" is_async="true" thread_priority="30">
       <hardware>
-        <plugin>drqp_control/a1_16_hardware_interface</plugin>
-        <param name="device_address">${device_address}</param>
-        <param name="baud_rate">115200</param>
+        <xacro:if value="${use_gazebo}">
+          <plugin>gz_ros2_control/GazeboSimSystem</plugin>
+        </xacro:if>
+        <xacro:unless value="${use_gazebo}">
+          <plugin>drqp_control/a1_16_hardware_interface</plugin>
+          <param name="device_address">${device_address}</param>
+          <param name="baud_rate">115200</param>
+        </xacro:unless>
       </hardware>
       <xacro:drqp_leg_ros2_control robot_name="${robot_name}" leg_name="left_front" coxa_servo_id="1"/>

Commit message: remove unused

File: packages/runtime/drqp_description/urdf/dr_qp.urdf.xacro (robot description, xacro)
@@ -6,7 +6,4 @@
   <material name="drqp_black">
     <texture filename="package://drqp_description/meshes/drqp_black.png"/>
-  </material>
-  <material name="drqp_black_tmp">
-    <color rgba="0.5 0.5 0.5 0.2" />
   </material>
   <xacro:property name="robot_height" value="0.085" />

Commit message: it is WORKING!!!! super slow though. physics setup might be way off

File: packages/runtime/drqp_description/urdf/dr_qp.urdf.xacro (robot description, xacro)
@@ -24,4 +24,6 @@
   <xacro:include filename="$(find drqp_description)/urdf/ros2_control.urdf.xacro"/>
   <xacro:drqp_ros2_control robot_name="$(arg robot_name)" device_address="$(arg hardware_device_address)" use_gazebo="$(arg use_gazebo)" />
+  <xacro:include filename="$(find drqp_description)/urdf/gazebo.xacro"/>
+  <xacro:gazebo />
   <gazebo reference="">
     <self_collide>1</self_collide>

File: packages/runtime/drqp_description/urdf/gazebo.xacro (robot description, xacro)
@@ -1,11 +1,11 @@
 <?xml version="1.0"?>
 <robot xmlns:xacro="http://www.ros.org/wiki/xacro">
-  <xacro:macro name="gazebo" params="robot_name">
-    <!-- Gazebo Classic definitions + plugin -->
-  <!-- <gazebo>
-    <plugin filename="gz_ros2_control-system" name="gz_ros2_control::GazeboSimROS2ControlPlugin">
-      <parameters>$(find drqp_control)/config/drqp_controllers.yaml</parameters>
-    </plugin>
-  </gazebo> -->
+  <xacro:macro name="gazebo">
+    <!-- ros_control plugin -->
+    <gazebo>
+      <plugin filename="gz_ros2_control-system" name="gz_ros2_control::GazeboSimROS2ControlPlugin">
+        <parameters>$(find drqp_control)/config/drqp_controllers.yml</parameters>
+      </plugin>
+    </gazebo>
   </xacro:macro>
 </robot>

Commit message: fix name

File: packages/runtime/drqp_description/urdf/dr_qp.urdf.xacro (robot description, xacro)
@@ -17,5 +17,5 @@
   <xacro:leg robot_name="$(arg robot_name)" prefix="right_back" x="-0.11692" y="-0.06387" yaw="${-3*pi/4}"/>
   <link name="world" />
-  <joint name="world_to_base_link=" type="fixed">
+  <joint name="world_to_base_link" type="fixed">
       <origin rpy="0 0 0" xyz="0 0 ${robot_height}"/>
       <parent link="world"/>

Commit message: rename world link to ground to

File: packages/runtime/drqp_description/urdf/dr_qp.urdf.xacro (robot description, xacro)
@@ -16,8 +16,8 @@
   <xacro:leg robot_name="$(arg robot_name)" prefix="left_back" x="-0.11692" y="0.06387" yaw="${3*pi/4}"/>
   <xacro:leg robot_name="$(arg robot_name)" prefix="right_back" x="-0.11692" y="-0.06387" yaw="${-3*pi/4}"/>
-  <link name="world" />
-  <joint name="world_to_base_link" type="fixed">
+  <link name="ground" />
+  <joint name="ground_to_base_link" type="fixed">
       <origin rpy="0 0 0" xyz="0 0 ${robot_height}"/>
-      <parent link="world"/>
+      <parent link="ground"/>
       <child link="$(arg robot_name)/base_link"/>
   </joint>
