Commit message: Migrate to modern gazebo (#244)
Migrate all dependencies to use modern gazebo and its bridge
Use `gz_ros2_control` for simulating servos
Migrate and fix URDF/SDF 

IT WORKS!!!
https://youtu.be/G6yNfmKsnHQ

---------

Co-authored-by: anton-matosov <3339485+anton-matosov@users.noreply.github.com>

File: packages/runtime/drqp_description/urdf/dr_qp.urdf.xacro (robot description, xacro)
@@ -2,19 +2,12 @@
 <robot name="dr_qp" xmlns:xacro="http://ros.org/wiki/xacro">
   <xacro:arg name="robot_name" default = "dr_qp"/>
-  <xacro:arg name="load_gazebo_configs" default="false"/>
   <xacro:arg name="hardware_device_address" default="/dev/ttySC0"/>
-  <xacro:if value="$(arg load_gazebo_configs)">
-    <xacro:include filename="$(find drqp_gazebo)/config/drqp_texture.gazebo"/>
-  </xacro:if>
+  <xacro:arg name="use_gazebo" default="false" />
   <material name="drqp_black">
     <texture filename="package://drqp_description/meshes/drqp_black.png"/>
-  </material>
-  <material name="drqp_black_tmp">
-    <color rgba="0.5 0.5 0.5 0.2" />
   </material>
   <xacro:property name="robot_height" value="0.085" />
   <xacro:include filename="$(find drqp_description)/urdf/body.urdf.xacro"/>
   <xacro:include filename="$(find drqp_description)/urdf/leg.urdf.xacro"/>
-  <!-- <xacro:include filename="$(find drqp_description)/urdf/gazebo.xacro"/> -->
   <xacro:leg robot_name="$(arg robot_name)" prefix="left_front" x="0.11692" y="0.06387" yaw="${pi/4}"/>
   <xacro:leg robot_name="$(arg robot_name)" prefix="right_front" x="0.11692" y="-0.06387" yaw="${-pi/4}"/>
@@ -23,14 +16,16 @@
   <xacro:leg robot_name="$(arg robot_name)" prefix="left_back" x="-0.11692" y="0.06387" yaw="${3*pi/4}"/>
   <xacro:leg robot_name="$(arg robot_name)" prefix="right_back" x="-0.11692" y="-0.06387" yaw="${-3*pi/4}"/>
-  <link name="world" />
-  <joint name="world_to_base_link=" type="fixed">
+  <link name="ground" />
+  <joint name="ground_to_base_link" type="fixed">
       <origin rpy="0 0 0" xyz="0 0 ${robot_height}"/>
-      <parent link="world"/>
+      <parent link="ground"/>
       <child link="$(arg robot_name)/base_link"/>
   </joint>
   <xacro:include filename="$(find drqp_description)/urdf/ros2_control.urdf.xacro"/>
-  <xacro:drqp_ros2_control robot_name="$(arg robot_name)" device_address="$(arg hardware_device_address)" />
-  <gazebo reference="">
-    <self_collide>1</self_collide>
+  <xacro:drqp_ros2_control robot_name="$(arg robot_name)" device_address="$(arg hardware_device_address)" use_gazebo="$(arg use_gazebo)" />
+  <xacro:include filename="$(find drqp_description)/urdf/gazebo.xacro"/>
+  <xacro:gazebo />
+  <gazebo>
+    <self_collide>true</self_collide>
     <!-- Params copied from https://www.youtube.com/watch?v=Gp3DF97yN7k&list=PL_0ePxMRfT22elbjPCf36MS02d6TK2sSk&index=1 -->
     <mu1>50</mu1>

File: packages/runtime/drqp_description/urdf/gazebo.xacro (robot description, xacro)
@@ -1,46 +1,11 @@
 <?xml version="1.0"?>
 <robot xmlns:xacro="http://www.ros.org/wiki/xacro">
-    <ros2_control name="GazeboSystem" type="system">
-        <!-- <hardware> Fix in https://github.com/Dr-QP/Dr.QP/issues/91
-            <plugin>gazebo_ros2_control/GazeboSystem</plugin>
-        </hardware> -->
-        <xacro:macro name="hexjoint" params="name">
-            <joint name="${name}">
-                <command_interface name="position">
-                    <param name="min">-15</param>
-                    <param name="max">15</param>
-                </command_interface>
-                <state_interface name="position">
-                    <param name="initial_value">1.0</param>
-                </state_interface>
-                <state_interface name="velocity" />
-                <state_interface name="effort" />
-            </joint>
-        </xacro:macro>
-        <xacro:hexjoint name="left_back_coxa" />
-        <xacro:hexjoint name="left_back_femur" />
-        <xacro:hexjoint name="left_back_tibia" />
-        <!-- <xacro:hexjoint name="left_middle_coxa" /> -->
-        <!-- <xacro:hexjoint name="left_middle_femur" /> -->
-        <!-- <xacro:hexjoint name="left_middle_tibia" /> -->
-        <!-- <xacro:hexjoint name="left_front_coxa" /> -->
-        <!-- <xacro:hexjoint name="left_front_femur" /> -->
-        <!-- <xacro:hexjoint name="left_front_tibia" /> -->
-        <!-- <xacro:hexjoint name="right_front_coxa" /> -->
-        <!-- <xacro:hexjoint name="right_front_femur" /> -->
-        <!-- <xacro:hexjoint name="right_front_tibia" /> -->
-        <!-- <xacro:hexjoint name="right_middle_coxa" /> -->
-        <!-- <xacro:hexjoint name="right_middle_femur" /> -->
-        <!-- <xacro:hexjoint name="right_middle_tibia" /> -->
-        <!-- <xacro:hexjoint name="right_back_coxa" /> -->
-        <!-- <xacro:hexjoint name="right_back_femur" /> -->
-        <!-- <xacro:hexjoint name="right_back_tibia" /> -->
-    </ros2_control>
-    <!-- <gazebo> Fix in https://github.com/Dr-QP/Dr.QP/issues/91
-        <plugin filename="libgazebo_ros2_control.so" name="gazebo_ros2_control">
-          <robot_param>robot_description</robot_param>
-          <robot_param_node>robot_state_publisher</robot_param_node>
-          <parameters>$(find drqp_gazebo)/config/gazebo_params.yaml</parameters>
-        </plugin>
-    </gazebo> -->
+  <xacro:macro name="gazebo">
+    <!-- ros_control plugin -->
+    <gazebo>
+      <plugin filename="gz_ros2_control-system" name="gz_ros2_control::GazeboSimROS2ControlPlugin">
+        <parameters>$(find drqp_control)/config/drqp_controllers.yml</parameters>
+      </plugin>
+    </gazebo>
+  </xacro:macro>
 </robot>

File: packages/runtime/drqp_description/urdf/leg.urdf.xacro (robot description, xacro)
@@ -9,12 +9,9 @@
   </xacro:macro>
   <xacro:macro name="leg" params="robot_name prefix x y yaw">
-  <joint name="${robot_name}/${prefix}_coxa_servo" type="fixed">
+  <joint name="${robot_name}/${prefix}_coxa_servo_joint" type="fixed">
     <origin rpy="0 0 ${yaw}" xyz="${x} ${y} 0"/>
     <parent link="${robot_name}/base_center_link"/>
     <child link="${robot_name}/${prefix}_coxa_servo"/>
   </joint>
-  <gazebo reference='${robot_name}/${prefix}_coxa_servo'>
-    <preserveFixedJoint>true</preserveFixedJoint>
-  </gazebo>
   <link name="${robot_name}/${prefix}_coxa_servo">
     <visual>
@@ -71,7 +68,4 @@
     <child link="${robot_name}/${prefix}_coxa_f2_link_2"/>
   </joint>
-  <gazebo reference='${robot_name}/${prefix}_coxa_inner'>
-    <preserveFixedJoint>true</preserveFixedJoint>
-  </gazebo>
   <link name="${robot_name}/${prefix}_coxa_f2_link_2">
     <visual>
@@ -133,7 +127,4 @@
     <child link="${robot_name}/${prefix}_femur_link_f3"/>
   </joint>
-  <gazebo reference='${robot_name}/${prefix}_femur_inner_1'>
-    <preserveFixedJoint>true</preserveFixedJoint>
-  </gazebo>
   <link name="${robot_name}/${prefix}_femur_link_f3">
     <visual>
@@ -161,7 +152,4 @@
     <child link="${robot_name}/${prefix}_femur_link_f1"/>
   </joint>
-  <gazebo reference='${robot_name}/${prefix}_femur_inner_2'>
-    <preserveFixedJoint>true</preserveFixedJoint>
-  </gazebo>
   <link name="${robot_name}/${prefix}_femur_link_f1">
     <visual>
@@ -219,12 +207,9 @@
     </inertial>
   </link>
-  <joint name="${robot_name}/${prefix}_tibia_leg" type="fixed">
+  <joint name="${robot_name}/${prefix}_tibia_leg_joint" type="fixed">
     <origin rpy="0 0 0" xyz="0.0325 0 0"/>
     <parent link="${robot_name}/${prefix}_tibia_servo"/>
     <child link="${robot_name}/${prefix}_tibia_leg"/>
   </joint>
-  <gazebo reference='${robot_name}/${prefix}_tibia_leg'>
-    <preserveFixedJoint>true</preserveFixedJoint>
-  </gazebo>
   <link name="${robot_name}/${prefix}_tibia_leg">
     <visual>
@@ -251,7 +236,4 @@
     <child link="${robot_name}/${prefix}_foot_link"/>
   </joint>
-  <gazebo reference='${robot_name}/${prefix}_foot'>
-    <preserveFixedJoint>true</preserveFixedJoint>
-  </gazebo>
   <link name="${robot_name}/${prefix}_foot_link"/>
 </xacro:macro>

File: packages/runtime/drqp_description/urdf/ros2_control.urdf.xacro (robot description, xacro)
@@ -48,10 +48,15 @@
     </joint>
   </xacro:macro>
-  <xacro:macro name="drqp_ros2_control" params="robot_name device_address:=/dev/ttySC0">
+  <xacro:macro name="drqp_ros2_control" params="robot_name device_address:=/dev/ttySC0 use_gazebo:=^|false">
     <ros2_control name="${robot_name}_servos" type="system" rw_rate="20" is_async="true" thread_priority="30">
       <hardware>
-        <plugin>drqp_control/a1_16_hardware_interface</plugin>
-        <param name="device_address">${device_address}</param>
-        <param name="baud_rate">115200</param>
+        <xacro:if value="${use_gazebo}">
+          <plugin>gz_ros2_control/GazeboSimSystem</plugin>
+        </xacro:if>
+        <xacro:unless value="${use_gazebo}">
+          <plugin>drqp_control/a1_16_hardware_interface</plugin>
+          <param name="device_address">${device_address}</param>
+          <param name="baud_rate">115200</param>
+        </xacro:unless>
       </hardware>
       <xacro:drqp_leg_ros2_control robot_name="${robot_name}" leg_name="left_front" coxa_servo_id="1"/>
