Commit message: add odometry publisher
Signed-off-by: Anton Matosov <anton.matosov@gmail.com>

File: packages/runtime/drqp_control/urdf/dr_qp.urdf.xacro (robot description, xacro)
@@ -26,5 +26,5 @@
   <xacro:if value="$(arg use_gazebo)">
     <xacro:include filename="$(find drqp_control)/urdf/gazebo.xacro"/>
-    <xacro:gazebo />
+    <xacro:gazebo robot_name="$(arg robot_name)" />
   </xacro:if>
   <gazebo>

File: packages/runtime/drqp_control/urdf/gazebo.xacro (robot description, xacro)
@@ -1,5 +1,5 @@
 <?xml version="1.0"?>
 <robot xmlns:xacro="http://www.ros.org/wiki/xacro">
-  <xacro:macro name="gazebo">
+  <xacro:macro name="gazebo" params="robot_name">
     <!-- ros_control plugin -->
     <gazebo>
@@ -7,4 +7,10 @@
         <parameters>$(find drqp_control)/config/drqp_controllers.yml</parameters>
       </plugin>
+      <plugin filename="gz-sim-odometry-publisher-system" name="gz::sim::systems::OdometryPublisher">
+        <odom_frame>odom</odom_frame>
+        <robot_base_frame>${robot_name}/base_link</robot_base_frame>
+        <odom_topic>/model/drqp/odometry</odom_topic>
+        <dimensions>3</dimensions>
+      </plugin>
     </gazebo>
   </xacro:macro>
