Commit message: Merge drqp_description into drqp_control package
Co-authored-by: anton-matosov <3339485+anton-matosov@users.noreply.github.com>

File: packages/runtime/drqp_control/urdf/body.urdf.xacro (robot description, xacro)
@@ -6,5 +6,5 @@
       <origin xyz="0 0 -${body_height/2}" rpy="${pi/2} 0 ${pi}" />
       <geometry>
-        <mesh filename="package://drqp_description/meshes/body-simple.stl" />
+        <mesh filename="package://drqp_control/meshes/body-simple.stl" />
       </geometry>
       <material name="drqp_black"/>
@@ -13,5 +13,5 @@
       <origin xyz="0 0 -${body_height/2}" rpy="0 0 0" />
       <geometry>
-        <mesh filename="package://drqp_description/meshes/body-collision.stl" />
+        <mesh filename="package://drqp_control/meshes/body-collision.stl" />
       </geometry>
     </collision>

File: packages/runtime/drqp_control/urdf/dr_qp.urdf.xacro (robot description, xacro)
@@ -5,9 +5,9 @@
   <xacro:arg name="use_gazebo" default="false" />
   <material name="drqp_black">
-    <texture filename="package://drqp_description/meshes/drqp_black.png"/>
+    <texture filename="package://drqp_control/meshes/drqp_black.png"/>
   </material>
   <xacro:property name="robot_height" value="0.085" />
-  <xacro:include filename="$(find drqp_description)/urdf/body.urdf.xacro"/>
-  <xacro:include filename="$(find drqp_description)/urdf/leg.urdf.xacro"/>
+  <xacro:include filename="$(find drqp_control)/urdf/body.urdf.xacro"/>
+  <xacro:include filename="$(find drqp_control)/urdf/leg.urdf.xacro"/>
   <xacro:leg robot_name="$(arg robot_name)" prefix="left_front" x="0.11692" y="0.06387" yaw="${pi/4}"/>
   <xacro:leg robot_name="$(arg robot_name)" prefix="right_front" x="0.11692" y="-0.06387" yaw="${-pi/4}"/>
@@ -22,7 +22,7 @@
       <child link="$(arg robot_name)/base_link"/>
   </joint>
-  <xacro:include filename="$(find drqp_description)/urdf/ros2_control.urdf.xacro"/>
+  <xacro:include filename="$(find drqp_control)/urdf/ros2_control.urdf.xacro"/>
   <xacro:drqp_ros2_control robot_name="$(arg robot_name)" device_address="$(arg hardware_device_address)" use_gazebo="$(arg use_gazebo)" />
-  <xacro:include filename="$(find drqp_description)/urdf/gazebo.xacro"/>
+  <xacro:include filename="$(find drqp_control)/urdf/gazebo.xacro"/>
   <xacro:gazebo />
   <gazebo>

File: packages/runtime/drqp_control/urdf/leg.urdf.xacro (robot description, xacro)
@@ -1,5 +1,5 @@
 <?xml version="1.0"?>
 <robot xmlns:xacro="http://ros.org/wiki/xacro">
-  <xacro:include filename="$(find drqp_description)/urdf/inertial_macros.xacro"/>
+  <xacro:include filename="$(find drqp_control)/urdf/inertial_macros.xacro"/>
   <xacro:macro name="inertial_stub" params="">
     <xacro:property name="tiny_value" value="0.01"/>
@@ -18,5 +18,5 @@
       <origin xyz="0 0 0" rpy="0 0 ${-pi/2}" />
       <geometry>
-        <mesh filename="package://drqp_description/meshes/servo.stl" />
+        <mesh filename="package://drqp_control/meshes/servo.stl" />
       </geometry>
       <material name="drqp_black"/>
@@ -25,5 +25,5 @@
       <origin xyz="0 0 0" rpy="0 0 ${-pi/2}" />
       <geometry>
-        <mesh filename="package://drqp_description/meshes/servo-collision.stl" />
+        <mesh filename="package://drqp_control/meshes/servo-collision.stl" />
       </geometry>
     </collision>
@@ -51,5 +51,5 @@
       <origin rpy="0 0 ${pi/2}" xyz="0 0 0"/>
       <geometry>
-        <mesh filename="package://drqp_description/meshes/F2.stl" />
+        <mesh filename="package://drqp_control/meshes/F2.stl" />
       </geometry>
       <material name="drqp_black"/>
@@ -58,5 +58,5 @@
       <origin rpy="0 0 ${pi/2}" xyz="0 0 0"/>
       <geometry>
-        <mesh filename="package://drqp_description/meshes/F2-collision.stl" />
+        <mesh filename="package://drqp_control/meshes/F2-collision.stl" />
       </geometry>
     </collision>
@@ -72,5 +72,5 @@
       <origin rpy="0 ${pi/2} ${-pi/2}" xyz="0 0 0"/>
       <geometry>
-        <mesh filename="package://drqp_description/meshes/F2.stl" />
+        <mesh filename="package://drqp_control/meshes/F2.stl" />
       </geometry>
       <material name="drqp_black"/>
@@ -79,5 +79,5 @@
       <origin rpy="0 ${pi/2} ${-pi/2}" xyz="0 0 0"/>
       <geometry>
-        <mesh filename="package://drqp_description/meshes/F2-collision.stl" />
+        <mesh filename="package://drqp_control/meshes/F2-collision.stl" />
       </geometry>
     </collision>
@@ -106,12 +106,12 @@
           36mm - distance from actuator center to the center of the holes on the back
          -->
-        <mesh filename="package://drqp_description/meshes/servo.stl" />
-      </geometry>
-      <material name="drqp_black"/>
-    </visual>
-    <collision>
-      <origin rpy="0 ${pi/2} ${pi/2}" xyz="0 0 0" />
-      <geometry>
-        <mesh filename="package://drqp_description/meshes/servo-collision.stl" />
+        <mesh filename="package://drqp_control/meshes/servo.stl" />
+      </geometry>
+      <material name="drqp_black"/>
+    </visual>
+    <collision>
+      <origin rpy="0 ${pi/2} ${pi/2}" xyz="0 0 0" />
+      <geometry>
+        <mesh filename="package://drqp_control/meshes/servo-collision.stl" />
       </geometry>
     </collision>
@@ -135,5 +135,5 @@
           5.5mm - distance from origin to center of the side mounting holes
          -->
-        <mesh filename="package://drqp_description/meshes/F3.stl" />
+        <mesh filename="package://drqp_control/meshes/F3.stl" />
       </geometry>
       <material name="drqp_black"/>
@@ -142,5 +142,5 @@
       <origin rpy="0 ${pi/2} ${pi/2}" xyz="0 0 0"/>
       <geometry>
-        <mesh filename="package://drqp_description/meshes/F3-collision.stl" />
+        <mesh filename="package://drqp_control/meshes/F3-collision.stl" />
       </geometry>
     </collision>
@@ -161,5 +161,5 @@
           23.0mm - distance from origin to mount plane - y axis
          -->
-        <mesh filename="package://drqp_description/meshes/F1.stl" />
+        <mesh filename="package://drqp_control/meshes/F1.stl" />
       </geometry>
       <material name="drqp_black"/>
@@ -168,5 +168,5 @@
       <origin rpy="${pi} ${-pi/2} ${pi/2}" xyz="0 0 0"/>
       <geometry>
-        <mesh filename="package://drqp_description/meshes/F1-collision.stl" />
+        <mesh filename="package://drqp_control/meshes/F1-collision.stl" />
       </geometry>
     </collision>
@@ -191,12 +191,12 @@
       <origin rpy="0 ${pi/2} ${pi/2}" xyz="0 0 0" />
       <geometry>
-        <mesh filename="package://drqp_description/meshes/servo.stl" />
-      </geometry>
-      <material name="drqp_black"/>
-    </visual>
-    <collision>
-      <origin rpy="0 ${pi/2} ${pi/2}" xyz="0 0 0" />
-      <geometry>
-        <mesh filename="package://drqp_description/meshes/servo-collision.stl" />
+        <mesh filename="package://drqp_control/meshes/servo.stl" />
+      </geometry>
+      <material name="drqp_black"/>
+    </visual>
+    <collision>
+      <origin rpy="0 ${pi/2} ${pi/2}" xyz="0 0 0" />
+      <geometry>
+        <mesh filename="package://drqp_control/meshes/servo-collision.stl" />
       </geometry>
     </collision>
@@ -219,5 +219,5 @@
           Origin is at end servo attachment, 32.5 between servo pivot and this point
          -->
-        <mesh filename="package://drqp_description/meshes/Tibia.stl" />
+        <mesh filename="package://drqp_control/meshes/Tibia.stl" />
       </geometry>
       <material name="drqp_black"/>
@@ -226,5 +226,5 @@
       <origin rpy="0 0 0" xyz="0 0 0"/>
       <geometry>
-        <mesh filename="package://drqp_description/meshes/Tibia-collision.stl" />
+        <mesh filename="package://drqp_control/meshes/Tibia-collision.stl" />
       </geometry>
     </collision>

Commit message: origin of attachment rotation is a joint prop
Signed-off-by: Anton Matosov <anton.matosov@gmail.com>

File: packages/runtime/drqp_control/urdf/body.urdf.xacro (robot description, xacro)
@@ -36,5 +36,5 @@
   </link>
   <joint name="base_center_to_imu" type="fixed">
-    <origin rpy="0 0 0" xyz="0.054633 0 0.103"/>
+    <origin rpy="${pi} 0 ${pi/2}" xyz="0.054633 0 0.103"/>
     <parent link="$(arg robot_name)/base_center_link"/>
     <child link="$(arg robot_name)/imu_link"/>
@@ -42,5 +42,4 @@
   <link name="$(arg robot_name)/imu_link">
      <visual>
-      <origin rpy="${pi} 0 ${pi/2}" xyz="0 0 0"/>
       <geometry>
           <!-- Chip footprint 3.8 mm x 5.2 mm, height 1.13 mm, X axis along short side -->
