Commit message: add chip size and orientation
Co-authored-by: Copilot <copilot@github.com>
Signed-off-by: Anton Matosov <anton.matosov@gmail.com>

File: packages/runtime/drqp_control/urdf/body.urdf.xacro (robot description, xacro)
@@ -36,9 +36,16 @@
   </link>
   <joint name="base_center_to_imu" type="fixed">
-    <origin rpy="0 0 0" xyz="0 0 0"/>
+    <origin rpy="0 0 0" xyz="0.054633 0 0.103"/>
     <parent link="$(arg robot_name)/base_center_link"/>
     <child link="$(arg robot_name)/imu_link"/>
   </joint>
   <link name="$(arg robot_name)/imu_link">
+    <!-- Footprint 3.8 mm x 5.2 mm, height 1.13 mm, X axis along short side -->
+     <visual>
+      <origin rpy="${pi} 0 ${pi/2}" xyz="0 0 0"/>
+      <geometry>
+          <box size="0.0038 0.0052 0.00113" />
+      </geometry>
+     </visual>
   </link>
 </robot>

Commit message: imu box
Co-authored-by: Copilot <copilot@github.com>
Signed-off-by: Anton Matosov <anton.matosov@gmail.com>

File: packages/runtime/drqp_control/urdf/body.urdf.xacro (robot description, xacro)
@@ -41,10 +41,13 @@
   </joint>
   <link name="$(arg robot_name)/imu_link">
-    <!-- Footprint 3.8 mm x 5.2 mm, height 1.13 mm, X axis along short side -->
      <visual>
       <origin rpy="${pi} 0 ${pi/2}" xyz="0 0 0"/>
       <geometry>
+          <!-- Chip footprint 3.8 mm x 5.2 mm, height 1.13 mm, X axis along short side -->
           <box size="0.0038 0.0052 0.00113" />
       </geometry>
+      <material name="imu_material">
+        <color rgba="0 1 1 1"/>
+      </material>
      </visual>
   </link>

Commit message: Rename dr_qp to drqp and improve IMU integration (#355)
# Summary

Rename the robot namespace and asset naming from `dr_qp` to `drqp`
across runtime, control, and simulation artifacts while continuing the
BNO055 IMU integration work. This branch also hardens IMU startup and
bridge behavior so hardware and Gazebo publish consistent frames and
topics with clearer failure modes.

## What Changed

- Standardized robot naming and frame or joint identifiers from `dr_qp`
to `drqp` across the workspace, including URDF/Xacro, configs, RViz,
trajectory builder logic, tests, and workspace settings.
- Finished the IMU integration by aligning the IMU link pose with the
robot model, relying on the node default `frame_id`, adding the BNO055
hardware dependencies (`adafruit-circuitpython-bno055`, `lgpio`), and
adding `scripts/bno.py` for direct sensor inspection.
- Hardened `drqp_brain.imu_node` by treating partial sensor vectors and
quaternions as unavailable, wrapping backend construction failures in
`SensorInitializationError`, and exiting `main()` cleanly with
actionable startup logs.
- Updated Gazebo bridge and control wiring so odometry and IMU topics
use the renamed robot namespace consistently while ROS-facing topics
remain on `/odom` and `/imu/data`; refreshed related tests and fixtures.
- Expanded `drqp_brain` tests to cover conversion helpers, backend
initialization failures, and CLI exit behavior.

## Why

Consistent `drqp` naming avoids controller, joint, and frame mismatches
between runtime, URDF, Gazebo, and tests. The IMU updates keep the
mounted sensor model aligned with published data and make bringup
failures easier to diagnose on real hardware or in mixed simulation
environments.

## How to Test

1. `source scripts/setup.bash --update-venv && python3 -m pytest
packages/runtime/drqp_brain/test/test_imu_node.py
packages/runtime/drqp_brain/test/test_joint_trajectory_builder.py -q`
2. Attempted broader validation with `source scripts/setup.bash
--update-venv && python3 -m pytest
packages/runtime/drqp_brain/test/test_imu_node.py
packages/runtime/drqp_brain/test/test_joint_trajectory_builder.py
packages/runtime/drqp_control/test/test_urdf.py
packages/runtime/drqp_control/test/test_a1_16_hardware_interface.py -q`
3. In this container, `packages/runtime/drqp_control/test/test_urdf.py`
failed while invoking `xacro` with `AttributeError: module 'xml' has no
attribute 'parsers'`, and
`packages/runtime/drqp_control/test/test_a1_16_hardware_interface.py`
failed because the required controller nodes were not running.

## Breaking Changes

- Renamed robot namespace, frame, and joint prefixes from `dr_qp` to
`drqp`.

## Migration

- Update any external launch, config, or test tooling that still
references `dr_qp/*` topics, frames, joints, or `dr_qp.urdf.xacro`.
- ROS-facing odometry consumers should use `/odom`; the Gazebo bridge
now sources odometry from `/model/drqp/odometry`.

---------

Signed-off-by: Anton Matosov <anton.matosov@gmail.com>
Co-authored-by: Copilot <copilot@github.com>
Co-authored-by: anton-matosov <3339485+anton-matosov@users.noreply.github.com>
Co-authored-by: Copilot Autofix powered by AI <175728472+Copilot@users.noreply.github.com>

File: packages/runtime/drqp_control/urdf/body.urdf.xacro (robot description, xacro)
@@ -1,4 +1,4 @@
 <?xml version="1.0"?>
-<robot name="dr_qp" xmlns:xacro="http://ros.org/wiki/xacro">
+<robot name="drqp" xmlns:xacro="http://ros.org/wiki/xacro">
   <xacro:property name="body_height" value="0.037" />
   <link name="$(arg robot_name)/base_center_link">
@@ -36,9 +36,18 @@
   </link>
   <joint name="base_center_to_imu" type="fixed">
-    <origin rpy="0 0 0" xyz="0 0 0"/>
+    <origin rpy="${pi} 0 ${pi/2}" xyz="0.054633 0 0.103"/>
     <parent link="$(arg robot_name)/base_center_link"/>
     <child link="$(arg robot_name)/imu_link"/>
   </joint>
   <link name="$(arg robot_name)/imu_link">
+     <visual>
+      <geometry>
+          <!-- Chip footprint 3.8 mm x 5.2 mm, height 1.13 mm, X axis along short side -->
+          <box size="0.0038 0.0052 0.00113" />
+      </geometry>
+      <material name="imu_material">
+        <color rgba="0 1 1 1"/>
+      </material>
+     </visual>
   </link>
 </robot>
