Commit message: fix gazebo hardware setup. it has to be sync
Signed-off-by: Anton Matosov <anton.matosov@gmail.com>

File: packages/runtime/drqp_control/urdf/ros2_control.urdf.xacro (robot description, xacro)
@@ -48,16 +48,5 @@
     </joint>
   </xacro:macro>
-  <xacro:macro name="drqp_ros2_control" params="robot_name device_address:=/dev/ttySC0 use_gazebo:=^|false">
-    <ros2_control name="${robot_name}_servos" type="system" rw_rate="20" is_async="true" thread_priority="30">
-      <hardware>
-        <xacro:if value="${use_gazebo}">
-          <plugin>gz_ros2_control/GazeboSimSystem</plugin>
-        </xacro:if>
-        <xacro:unless value="${use_gazebo}">
-          <plugin>drqp_control/a1_16_hardware_interface</plugin>
-          <param name="device_address">${device_address}</param>
-          <param name="baud_rate">115200</param>
-        </xacro:unless>
-      </hardware>
+  <xacro:macro name="drqp_ros2_control_interfaces" params="robot_name">
       <xacro:drqp_leg_ros2_control robot_name="${robot_name}" leg_name="left_front" coxa_servo_id="1"/>
       <xacro:drqp_leg_ros2_control robot_name="${robot_name}" leg_name="right_front" coxa_servo_id="2" servo_inverted="True"/>
@@ -74,5 +63,24 @@
         </state_interface>
       </sensor>
-    </ros2_control>
+  </xacro:macro>
+  <xacro:macro name="drqp_ros2_control" params="robot_name device_address:=/dev/ttySC0 use_gazebo:=^|false">
+    <xacro:if value="${use_gazebo}">
+      <ros2_control name="${robot_name}_servos" type="system">
+        <hardware>
+          <plugin>gz_ros2_control/GazeboSimSystem</plugin>
+        </hardware>
+        <xacro:drqp_ros2_control_interfaces robot_name="${robot_name}"/>
+      </ros2_control>
+    </xacro:if>
+    <xacro:unless value="${use_gazebo}">
+      <ros2_control name="${robot_name}_servos" type="system" rw_rate="20" is_async="true" thread_priority="30">
+        <hardware>
+          <plugin>drqp_control/a1_16_hardware_interface</plugin>
+          <param name="device_address">${device_address}</param>
+          <param name="baud_rate">115200</param>
+        </hardware>
+        <xacro:drqp_ros2_control_interfaces robot_name="${robot_name}"/>
+      </ros2_control>
+    </xacro:unless>
   </xacro:macro>
 </robot>
